File: hw/teacup-carrier.kicad_sch (KiCad schematic)
At the start: 80 parts, among them J1 AH58893-T9B10-3F, J2 TYPE-C-31-M-12, J3 TE_292303-7, J4 Hirose_DM3D-SF, J5 Wuerth_694106301002, J6 AudioJack4_Ground, J7 SFW15R-2STE1LF, J8 SFW15R-2STE1LF, J9 TYPE-C-31-M-12, Q1 AO3401A, Q2 AO3401A, SW1 SSSS711403, SW2 SSSS711403, U1 AP62600SJ-7, U10 TS5A3166, U11 DIP-8 Socket, U12 TPS2053BDR, U13 W25Q32JVSS, U14 TPS22990DMLR, U15 TCA9555PWR, U2 AP62300WU-7, U3 MCP4661-104E_ST, U4 TPS22990DMLR, U5 AZ1117CH-3.3TRG1, U6 AZ1117CH-1.8TRG1, U7 AP62300WU-7, U8 ESP32-S3-WROOM-1-N16R2, U9 TS5A3166

Commit message: Carrier board: pin-breakout header sheet (SS8 superset)
Assigns J1 pins 87-169 (previously RESERVED_P87-96 and unconnected)
to the per-SoC GPIO/peripheral superset and breaks them out onto 11
function-clustered, labeled 0.1" headers on a new headers.kicad_sch
sheet: GMAC0/GMAC1 (RGMII, A1's real 2nd MAC), UART0/UART2/UART3
(no UART4/UART5 -- verified no T-series/A1 SoC has them), SSI0, SSI1,
PWM0-7, SAR-ADC, general SMB0/SMB1 (isolated from the carrier-ID I2C
bus), and 16 plain GPIO. Clustering is a silkscreen convenience only,
not an electrical constraint.

Verified: 0 layout overlaps, netlist diff shows only J1 pins 87-169
and the new header refs changed, ERC errors went down (231->158,
purely fewer not-connected pins) with no new violation classes.

Also commits the schematic generator toolchain (hw/scripts/) that
built this and the previously-merged power/connector/bmc/io sections,
so the schematic has a reproducible source instead of only generated
output.
Parts:
- added J20: HDR_J20, Connector_PinHeader_2.54mm:PinHeader_1x11_P2.54mm_Vertical, symbol Connector_Generic:Conn_01x11
- added J21: HDR_J21, Connector_PinHeader_2.54mm:PinHeader_1x11_P2.54mm_Vertical, symbol Connector_Generic:Conn_01x11
- added J22: HDR_J22, Connector_PinHeader_2.54mm:PinHeader_1x05_P2.54mm_Vertical, symbol Connector_Generic:Conn_01x05
- added J23: HDR_J23, Connector_PinHeader_2.54mm:PinHeader_1x05_P2.54mm_Vertical, symbol Connector_Generic:Conn_01x05
- added J24: HDR_J24, Connector_PinHeader_2.54mm:PinHeader_1x05_P2.54mm_Vertical, symbol Connector_Generic:Conn_01x05
- added J25: HDR_J25, Connector_PinHeader_2.54mm:PinHeader_1x07_P2.54mm_Vertical, symbol Connector_Generic:Conn_01x07
- added J26: HDR_J26, Connector_PinHeader_2.54mm:PinHeader_1x05_P2.54mm_Vertical, symbol Connector_Generic:Conn_01x05
- added J27: HDR_J27, Connector_PinHeader_2.54mm:PinHeader_1x09_P2.54mm_Vertical, symbol Connector_Generic:Conn_01x09
- added J28: HDR_J28, Connector_PinHeader_2.54mm:PinHeader_1x02_P2.54mm_Vertical, symbol Connector_Generic:Conn_01x02
- added J29: HDR_J29, Connector_PinHeader_2.54mm:PinHeader_1x05_P2.54mm_Vertical, symbol Connector_Generic:Conn_01x05
- added J30: HDR_J30, Connector_PinHeader_2.54mm:PinHeader_1x17_P2.54mm_Vertical, symbol Connector_Generic:Conn_01x17
Connections:
- net GND: now also J1.102 (P102), J1.107 (P107), J1.112 (P112), J1.123 (P123), J1.130 (P130), J1.135 (P135), J1.144 (P144), J1.145 (P145), J1.147 (P147), J1.152 (P152), J1.169 (P169), J1.97 (P97), J20.1 (Pin_1), J21.1 (Pin_1), J22.1 (Pin_1), J23.1 (Pin_1), J24.1 (Pin_1), J25.1 (Pin_1), J26.1 (Pin_1), J27.1 (Pin_1), J28.1 (Pin_1), J29.1 (Pin_1), J30.1 (Pin_1)
- net SAR_AUX0: now reaches J1.146 (P146)
- net SAR_AUX0: now also J28.2 (Pin_2)
- net SMB0_SDA: now reaches J1.148 (P148)
- net SMB0_SDA: now also J29.2 (Pin_2)
- net SMB0_SCK: now reaches J1.149 (P149)
- net SMB0_SCK: now also J29.3 (Pin_3)
- net SMB1_SDA: now reaches J1.150 (P150)
- net SMB1_SDA: now also J29.4 (Pin_4)
- net SMB1_SCK: now reaches J1.151 (P151)
- net SMB1_SCK: now also J29.5 (Pin_5)
- net GPIO0: now reaches J1.153 (P153)
- net GPIO0: now also J30.2 (Pin_2)
- net GPIO1: now reaches J1.154 (P154)
- net GPIO1: now also J30.3 (Pin_3)
- net GPIO2: now reaches J1.155 (P155)
- net GPIO2: now also J30.4 (Pin_4)
- net GPIO3: now reaches J1.156 (P156)
- net GPIO3: now also J30.5 (Pin_5)
- net GPIO4: now reaches J1.157 (P157)
- net GPIO4: now also J30.6 (Pin_6)
- net GPIO5: now reaches J1.158 (P158)
- net GPIO5: now also J30.7 (Pin_7)
- net GPIO6: now reaches J1.159 (P159)
- net GPIO6: now also J30.8 (Pin_8)
- net GPIO7: now reaches J1.160 (P160)
- net GPIO7: now also J30.9 (Pin_9)
- net GPIO8: now reaches J1.161 (P161)
- net GPIO8: now also J30.10 (Pin_10)
- net GPIO9: now reaches J1.162 (P162)
- net GPIO9: now also J30.11 (Pin_11)
- net GPIO10: now reaches J1.163 (P163)
- net GPIO10: now also J30.12 (Pin_12)
- net GPIO11: now reaches J1.164 (P164)
- net GPIO11: now also J30.13 (Pin_13)
- net GPIO12: now reaches J1.165 (P165)
- net GPIO12: now also J30.14 (Pin_14)
- net GPIO13: now reaches J1.166 (P166)
- net GPIO13: now also J30.15 (Pin_15)
- net GPIO14: now reaches J1.167 (P167)
- net GPIO14: now also J30.16 (Pin_16)
- net GPIO15: now reaches J1.168 (P168)
- net GPIO15: now also J30.17 (Pin_17)
- net UART0_CTS: now reaches J1.100 (P100)
- net UART0_CTS: now also J22.4 (Pin_4)
- net UART0_RTS: now reaches J1.101 (P101)
- net UART0_RTS: now also J22.5 (Pin_5)
- net UART2_RXD: now reaches J1.103 (P103)
- net UART2_RXD: now also J23.2 (Pin_2)
- net UART2_TXD: now reaches J1.104 (P104)
- net UART2_TXD: now also J23.3 (Pin_3)
- net UART2_CTS: now reaches J1.105 (P105)
- net UART2_CTS: now also J23.4 (Pin_4)
- net UART2_RTS: now reaches J1.106 (P106)
- net UART2_RTS: now also J23.5 (Pin_5)
- net UART3_RXD: now reaches J1.108 (P108)
- net UART3_RXD: now also J24.2 (Pin_2)
- net UART3_TXD: now reaches J1.109 (P109)
- net UART3_TXD: now also J24.3 (Pin_3)
- net UART3_CTS: now reaches J1.110 (P110)
- net UART3_CTS: now also J24.4 (Pin_4)
- net UART3_RTS: now reaches J1.111 (P111)
- net UART3_RTS: now also J24.5 (Pin_5)
- net GMAC1_MDIO: now reaches J1.113 (P113)
- net GMAC1_MDIO: now also J21.2 (Pin_2)
- net GMAC1_MDCK: now reaches J1.114 (P114)
- net GMAC1_MDCK: now also J21.3 (Pin_3)
- net GMAC1_TXCLK: now reaches J1.115 (P115)
- net GMAC1_TXCLK: now also J21.4 (Pin_4)
- net GMAC1_PHYCLK: now reaches J1.116 (P116)
- net GMAC1_PHYCLK: now also J21.5 (Pin_5)
- net GMAC1_TXEN: now reaches J1.117 (P117)
- net GMAC1_TXEN: now also J21.6 (Pin_6)
- net GMAC1_TXD0: now reaches J1.118 (P118)
- net GMAC1_TXD0: now also J21.7 (Pin_7)
- net GMAC1_TXD1: now reaches J1.119 (P119)
- net GMAC1_TXD1: now also J21.8 (Pin_8)
- net GMAC1_RXDV: now reaches J1.120 (P120)
- net GMAC1_RXDV: now also J21.9 (Pin_9)
- net GMAC1_RXD0: now reaches J1.121 (P121)
- net GMAC1_RXD0: now also J21.10 (Pin_10)
- net GMAC1_RXD1: now reaches J1.122 (P122)
- net GMAC1_RXD1: now also J21.11 (Pin_11)
- net SSI0_CLK: now reaches J1.124 (P124)
- net SSI0_CLK: now also J25.2 (Pin_2)
- net SSI0_DT: now reaches J1.125 (P125)
- net SSI0_DT: now also J25.3 (Pin_3)
- net SSI0_DR: now reaches J1.126 (P126)
- net SSI0_DR: now also J25.4 (Pin_4)
- net SSI0_CE0: now reaches J1.127 (P127)
- net SSI0_CE0: now also J25.5 (Pin_5)
- net SSI0_CE1: now reaches J1.128 (P128)
- net SSI0_CE1: now also J25.6 (Pin_6)
- net SSI0_GPC: now reaches J1.129 (P129)
- net SSI0_GPC: now also J25.7 (Pin_7)
- net SSI1_CLK: now reaches J1.131 (P131)
- net SSI1_CLK: now also J26.2 (Pin_2)
- net SSI1_DT: now reaches J1.132 (P132)
- net SSI1_DT: now also J26.3 (Pin_3)
- net SSI1_DR: now reaches J1.133 (P133)
- net SSI1_DR: now also J26.4 (Pin_4)
- net SSI1_CE0: now reaches J1.134 (P134)
- net SSI1_CE0: now also J26.5 (Pin_5)
- net PWM0: now reaches J1.136 (P136)
- net PWM0: now also J27.2 (Pin_2)
- net PWM1: now reaches J1.137 (P137)
- net PWM1: now also J27.3 (Pin_3)
- net PWM2: now reaches J1.138 (P138)
- net PWM2: now also J27.4 (Pin_4)
- net PWM3: now reaches J1.139 (P139)
- net PWM3: now also J27.5 (Pin_5)
- net PWM4: now reaches J1.140 (P140)
- net PWM4: now also J27.6 (Pin_6)
- net PWM5: now reaches J1.141 (P141)
- net PWM5: now also J27.7 (Pin_7)
- net PWM6: now reaches J1.142 (P142)
- net PWM6: now also J27.8 (Pin_8)
- net PWM7: now reaches J1.143 (P143)
- net PWM7: now also J27.9 (Pin_9)
- net UART0_RXD: now reaches J1.98 (P98)
- net UART0_RXD: now also J22.2 (Pin_2)
- net UART0_TXD: now reaches J1.99 (P99)
- net UART0_TXD: now also J22.3 (Pin_3)
- net RESERVED_P87 renamed GMAC0_MDIO
- net GMAC0_MDIO: now also J20.2 (Pin_2)
- net RESERVED_P88 renamed GMAC0_MDCK
- net GMAC0_MDCK: now also J20.3 (Pin_3)
- net RESERVED_P89 renamed GMAC0_TXCLK
- net GMAC0_TXCLK: now also J20.4 (Pin_4)
- net RESERVED_P90 renamed GMAC0_PHYCLK
- net GMAC0_PHYCLK: now also J20.5 (Pin_5)
- net RESERVED_P91 renamed GMAC0_TXEN
- net GMAC0_TXEN: now also J20.6 (Pin_6)
- net RESERVED_P92 renamed GMAC0_TXD0
- net GMAC0_TXD0: now also J20.7 (Pin_7)
- net RESERVED_P93 renamed GMAC0_TXD1
- net GMAC0_TXD1: now also J20.8 (Pin_8)
- net RESERVED_P94 renamed GMAC0_RXDV
- net GMAC0_RXDV: now also J20.9 (Pin_9)
- net RESERVED_P95 renamed GMAC0_RXD0
- net GMAC0_RXD0: now also J20.10 (Pin_10)
- net RESERVED_P96 renamed GMAC0_RXD1
- net GMAC0_RXD1: now also J20.11 (Pin_11)
Other:
- note added: "GMAC0 (RGMII0)"
- note added: "GMAC1 (RGMII1, A1 2nd MAC)"
- note added: "GPIO0-15 (plain)"
- note added: "PIN BREAKOUT HEADERS"
- note added: "PWM0-7"
- note added: "SAR-ADC"
- note added: "SMB0/SMB1 (general I2C)"
- note added: "SSI0 (SPI master)"
- note added: "SSI1"
- note added: "UART0"
- note added: "UART2"
- note added: "UART3"
- moved on the sheet: C1, C10, C11, C12, C13, C14, C15, C16, C17, C18, C19, C2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
