File: hw/teacup-carrier.kicad_sch (KiCad schematic)
At the start: 134 parts, among them J1 AH58893-T9B10-3F, J2 TYPE-C-31-M-12, J20 HDR_J20, J21 HDR_J21, J22 HDR_J22, J23 HDR_J23, J24 HDR_J24, J25 HDR_J25, J26 HDR_J26, J27 HDR_J27, J28 HDR_J28, J29 HDR_J29, J3 TE_292303-7, J30 HDR_J30, J31 HDR_J31, J32 HDR_J32, J33 HDR_J33, J34 HDR_J34, J35 HDR_J35, J36 HDR_J36, J37 HDR_J37, J38 AMP_MIC_TAP, J4 Hirose_DM3D-SF, J5 Wuerth_694106301002, J6 AudioJack4_Ground, J7 SFW15R-2STE1LF, J8 SFW15R-2STE1LF, J9 TYPE-C-31-M-12, Q1 AO3401A, Q2 AO3401A, SW1 SSSS711403, SW2 SSSS711403, U1 AP62600SJ-7, U10 TS5A3166, U11 DIP-8 Socket, U12 TPS2053BDR, U13 W25Q32JVSS, U14 TPS22990DMLR, U15 TCA9555PWR, U2 AP62300WU-7, U3 MCP4661-104E_ST, U4 TPS22990DMLR, U5 AZ1117CH-3.3TRG1, U6 AZ1117CH-1.8TRG1, U7 AP62300WU-7, U8 ESP32-S3-WROOM-1-N16R2, U9 TS5A3166

Commit message: Backfill MPN/Manufacturer fields on carrier and interposer schematics
Placed symbol instances only carried Reference/Value/Footprint; MPN and
Manufacturer were never propagated from the library cache, so BOM export
had a blank MPN column for every part. Fills in MPN (and Manufacturer
where unambiguous) for the 32 parts whose Value string is already a real
manufacturer part number - ICs, diodes, MOSFETs, switches, and specific
connectors - across the carrier, T31ZX interposer, and T41 interposer.
Generic passives, headers, and jumpers are left untouched since their
Value is a spec, not a part number.

ERC-neutral: 426/175/169 violations before and after on the three files.
Parts:
- D1, D2: MPN (none) -> PMEG2010ER; Manufacturer (none) -> Nexperia
- J2, J9: MPN (none) -> TYPE-C-31-M-12; Manufacturer (none) -> Hroparts Elec
- J3: MPN (none) -> 292303-7; Manufacturer (none) -> TE Connectivity
- J4: MPN (none) -> DM3D-SF; Manufacturer (none) -> Hirose Electric
- J5: MPN (none) -> 694106301002; Manufacturer (none) -> Wurth Elektronik
- J7, J8: MPN (none) -> SFW15R-2STE1LF; Manufacturer (none) -> JAE Electronics
- Q1, Q2: MPN (none) -> AO3401A; Manufacturer (none) -> Alpha & Omega Semiconductor
- SW1, SW2: MPN (none) -> SSSS711403
- U1: MPN (none) -> AP62600SJ-7; Manufacturer (none) -> Diodes Incorporated
- U10, U9: MPN (none) -> TS5A3166; Manufacturer (none) -> Texas Instruments
- U12: MPN (none) -> TPS2053BDR; Manufacturer (none) -> Texas Instruments
- U13: MPN (none) -> W25Q32JVSS; Manufacturer (none) -> Winbond Electronics
- U14, U4: MPN (none) -> TPS22990DMLR; Manufacturer (none) -> Texas Instruments
- U15: MPN (none) -> TCA9555PWR; Manufacturer (none) -> Texas Instruments
- U2, U7: MPN (none) -> AP62300WU-7; Manufacturer (none) -> Diodes Incorporated
- U3: MPN (none) -> MCP4661-104E/ST; Manufacturer (none) -> Microchip Technology
- U5: MPN (none) -> AZ1117CH-3.3TRG1
- U6: MPN (none) -> AZ1117CH-1.8TRG1
- U8: MPN (none) -> ESP32-S3-WROOM-1-N16R2; Manufacturer (none) -> Espressif Systems
