File: hw/teacup-carrier.kicad_sch (KiCad schematic)
At the start: 133 parts, among them J1 AH58893-T9B10-3F, J2 TYPE-C-31-M-12, J20 HDR_J20, J21 HDR_J21, J22 HDR_J22, J23 HDR_J23, J24 HDR_J24, J25 HDR_J25, J26 HDR_J26, J27 HDR_J27, J28 HDR_J28, J29 HDR_J29, J3 TE_292303-7, J30 HDR_J30, J31 HDR_J31, J32 HDR_J32, J33 HDR_J33, J34 HDR_J34, J35 HDR_J35, J36 HDR_J36, J37 HDR_J37, J38 AMP_MIC_TAP, J4 Hirose_DM3D-SF, J5 Wuerth_694106301002, J6 AudioJack4_Ground, J7 SFW15R-2STE1LF, J8 SFW15R-2STE1LF, J9 TYPE-C-31-M-12, Q1 AO3401A, Q2 AO3401A, SW1 SSSS711403, SW2 SSSS711403, U1 AP62600SJ-7, U10 TS5A3166, U11 DIP-8 Socket, U12 TPS2053BDR, U13 W25Q32JVSS, U14 TPS22990DMLR, U15 TCA9555PWR, U2 AP62300WU-7, U3 MCP4661-104E_ST, U4 TPS22990DMLR, U5 AZ1117CH-3.3TRG1, U6 AZ1117CH-1.8TRG1, U7 AP62300WU-7, U8 ESP32-S3-WROOM-1-N16R2, U9 TS5A3166

Commit message: Fix schematic<->PCB linking, reorder J1 pins by connected peer, add +3V3 plane, wire microSD card-detect
- schgen.py: deterministic per-symbol UUIDs (uuid5, keyed on ref designator)
  instead of random uuid4, so PCB footprints stay linked to their schematic
  symbol across regenerations; link all 133 real PCB footprints to their
  schematic symbol via path, fixing "Update PCB from Schematic" placing
  duplicates.
- J1 pin reorg: audio (HPOUTL/MICLP) moved from 170/171 to 6/7 (170/171 now
  GND); USBA_HOST_DP/DM moved from 40/41 to 20/21 (40/41 now GND); the 20
  pins connected directly to U8 (ESP32-S3) reordered so U8's ascending pin
  number maps to J1's descending pin number; +5V_MODEA (redundant -- a
  self-contained module already needs its own bare-bench power input)
  replaced with +5V_SW (the real arbitrated switched-5V rail) on pins 17/18.
- New +3V3 copper pour on In1.Cu, mirroring the existing GND pour; every
  +3V3 pad on the board (38, now 39 with R43) gets a stub trace + via down
  to it.
- microSD (J4): switched to the Micro_SD_Card_Det2 symbol so pin 10 (the
  footprint's real card-detect pad) has somewhere to attach; added R43
  (1M, matches TeaCup 3.3's R22) pulling MSC0_CD up to +3V3.
- fp-lib-table: replaced hardcoded /usr/share/kicad/footprints/... paths
  with ${KICAD10_FOOTPRINT_DIR}, fixing "footprint not found" errors for
  every component when Update PCB from Schematic runs outside this Linux
  environment.

Verified throughout via isolated ERC/DRC diffs against pre-change
baselines; each change confirmed to produce only its own intended delta.
Parts:
- removed unit 1 of J1
- removed unit 2 of J1
- removed unit 4 of J1
- removed unit 3 of J1
- removed unit 5 of J1
- removed J4: Hirose_DM3D-SF, Connector_Card:microSD_HC_Hirose_DM3D-SF, symbol Connector:Micro_SD_Card
- added J4: Hirose_DM3D-SF, Connector_Card:microSD_HC_Hirose_DM3D-SF, symbol Connector:Micro_SD_Card_Det2
- added R43: 1M, Resistor_SMD:R_0402_1005Metric, symbol Device:R
Connections:
- net +1V8: now also J1.15 (P15), J1.16 (P16)
- net +3V3: now also J1.13 (P13), J1.14 (P14), J4.4 (VDD), R43.1
- net +5V_SW: now also J1.17 (P17), J1.18 (P18)
- net BOOTSEL: now also J1.35 (P35)
- net GMAC0_MDCK: now also J1.88 (P88)
- net GMAC0_MDIO: now also J1.87 (P87)
- net GMAC0_PHYCLK: now also J1.90 (P90)
- net GMAC0_RXD0: now also J1.95 (P95)
- net GMAC0_RXD1: now also J1.96 (P96)
- net GMAC0_RXDV: now also J1.94 (P94)
- net GMAC0_TXCLK: now also J1.89 (P89)
- net GMAC0_TXD0: now also J1.92 (P92)
- net GMAC0_TXD1: now also J1.93 (P93)
- net GMAC0_TXEN: now also J1.91 (P91)
- net GMAC1_MDCK: now also J1.114 (P114)
- net GMAC1_MDIO: now also J1.113 (P113)
- net GMAC1_PHYCLK: now also J1.116 (P116)
- net GMAC1_RXD0: now also J1.121 (P121)
- net GMAC1_RXD1: now also J1.122 (P122)
- net GMAC1_RXDV: now also J1.120 (P120)
- net GMAC1_TXCLK: now also J1.115 (P115)
- net GMAC1_TXD0: now also J1.118 (P118)
- net GMAC1_TXD1: now also J1.119 (P119)
- net GMAC1_TXEN: now also J1.117 (P117)
- net GND: now also J1.102 (P102), J1.107 (P107), J1.11 (P11), J1.112 (P112), J1.12 (P12), J1.123 (P123), J1.130 (P130), J1.135 (P135), J1.144 (P144), J1.145 (P145), J1.147 (P147), J1.152 (P152), J1.169 (P169), J1.170 (P170), J1.171 (P171), J1.172 (P172), J1.19 (P19), J1.22 (P22), J1.36 (P36), J1.37 (P37), J1.38 (P38), J1.39 (P39), J1.40 (P40), J1.41 (P41), J1.49 (P49), J1.5 (P5), J1.51 (P51), J1.57 (P57), J1.58 (P58), J1.59 (P59), J1.63 (P63), J1.66 (P66), J1.69 (P69), J1.72 (P72), J1.76 (P76), J1.79 (P79), J1.8 (P8), J1.82 (P82), J1.85 (P85), J1.86 (P86), J1.97 (P97), J4.6 (VSS), J4.9 (DET_B)
- net GPIO0: now also J1.153 (P153)
- net GPIO1: now also J1.154 (P154)
- net GPIO10: now also J1.163 (P163)
- net GPIO11: now also J1.164 (P164)
- net GPIO12: now also J1.165 (P165)
- net GPIO13: now also J1.166 (P166)
- net GPIO14: now also J1.167 (P167)
- net GPIO15: now also J1.168 (P168)
- net GPIO2: now also J1.155 (P155)
- net GPIO3: now also J1.156 (P156)
- net GPIO4: now also J1.157 (P157)
- net GPIO5: now also J1.158 (P158)
- net GPIO6: now also J1.159 (P159)
- net GPIO7: now also J1.160 (P160)
- net GPIO8: now also J1.161 (P161)
- net GPIO9: now also J1.162 (P162)
- net HOSTED_DATA_READY: now also J1.24 (P24)
- net HOSTED_HANDSHAKE: now also J1.25 (P25)
- net HOSTED_RESET: now also J1.48 (P48)
- net HOSTED_SPI_CLK: now also J1.45 (P45)
- net HOSTED_SPI_CS: now also J1.26 (P26)
- net HOSTED_SPI_MISO: now also J1.27 (P27)
- net HOSTED_SPI_MOSI: now also J1.44 (P44)
- net HPOUTL: now also J1.7 (P7)
- net I2C_ID_SCL: now also J1.46 (P46)
- net I2C_ID_SDA: now also J1.47 (P47)
- net MICLP: now also J1.6 (P6)
- net MIPI0_CLKN: now also J1.65 (P65)
- net MIPI0_CLKP: now also J1.64 (P64)
- net MIPI0_D0N: now also J1.71 (P71)
- net MIPI0_D0P: now also J1.70 (P70)
- net MIPI0_D1N: now also J1.68 (P68)
- net MIPI0_D1P: now also J1.67 (P67)
- net MIPI0_GPIO: now also J1.62 (P62)
- net MIPI0_SCCB_SCL: now also J1.61 (P61)
- net MIPI0_SCCB_SDA: now also J1.60 (P60)
- net MIPI1_CLKN: now also J1.78 (P78)
- net MIPI1_CLKP: now also J1.77 (P77)
- net MIPI1_D0N: now also J1.84 (P84)
- net MIPI1_D0P: now also J1.83 (P83)
- net MIPI1_D1N: now also J1.81 (P81)
- net MIPI1_D1P: now also J1.80 (P80)
- net MIPI1_GPIO: now also J1.75 (P75)
- net MIPI1_SCCB_SCL: now also J1.74 (P74)
- net MIPI1_SCCB_SDA: now also J1.73 (P73)
- net MSC0_CLK: now also J1.53 (P53), J4.5 (CLK)
- net MSC0_CMD: now also J1.54 (P54), J4.3 (CMD)
- net MSC0_D0: now also J1.52 (P52), J4.7 (DAT0)
- net MSC0_D1: now also J1.50 (P50), J4.8 (DAT1)
- net MSC0_D2: now also J1.56 (P56), J4.1 (DAT2)
- net MSC0_D3_CD: now also J1.55 (P55), J4.2 (DAT3/CD)
- net PWM0: now also J1.136 (P136)
- net PWM1: now also J1.137 (P137)
- net PWM2: now also J1.138 (P138)
- net PWM3: now also J1.139 (P139)
- net PWM4: now also J1.140 (P140)
- net PWM5: now also J1.141 (P141)
- net PWM6: now also J1.142 (P142)
- net PWM7: now also J1.143 (P143)
- net RESET_EN: now also J1.34 (P34)
- net SAR_AUX0: now also J1.146 (P146)
- net SFC_CLK: now also J1.30 (P30)
- net SFC_CS: now also J1.32 (P32)
- net SFC_IO0: now also J1.31 (P31)
- net SFC_IO1: now also J1.29 (P29)
- net SFC_IO2: now also J1.28 (P28)
- net SFC_IO3: now also J1.33 (P33)
- net SMB0_SCK: now also J1.149 (P149)
- net SMB0_SDA: now also J1.148 (P148)
- net SMB1_SCK: now also J1.151 (P151)
- net SMB1_SDA: now also J1.150 (P150)
- net SPARE_P173: now also J1.173 (P173)
- net SPARE_P174: now also J1.174 (P174)
- net SPARE_P175: now also J1.175 (P175)
- net SPARE_P176: now also J1.176 (P176)
- net SPARE_P177: now also J1.177 (P177)
- net SPARE_P178: now also J1.178 (P178)
- net SPARE_P179: now also J1.179 (P179)
- net SPARE_P180: now also J1.180 (P180)
- net SPARE_P181: now also J1.181 (P181)
- net SPARE_P182: now also J1.182 (P182)
- net SPARE_P183: now also J1.183 (P183)
- net SPARE_P184: now also J1.184 (P184)
- net SPARE_P185: now also J1.185 (P185)
- net SPARE_P186: now also J1.186 (P186)
- net SPARE_P187: now also J1.187 (P187)
- net SPARE_P188: now also J1.188 (P188)
- net SPARE_P189: now also J1.189 (P189)
- net SPARE_P190: now also J1.190 (P190)
- net SPARE_P191: now also J1.191 (P191)
- net SPARE_P192: now also J1.192 (P192)
- net SPARE_P193: now also J1.193 (P193)
- net SPARE_P194: now also J1.194 (P194)
- net SPARE_P195: now also J1.195 (P195)
- net SPARE_P196: now also J1.196 (P196)
- net SPARE_P197: now also J1.197 (P197)
- net SPARE_P198: now also J1.198 (P198)
- net SPARE_P199: now also J1.199 (P199)
- net SPARE_P200: now also J1.200 (P200)
- net SPARE_P201: now also J1.201 (P201)
- net SPARE_P202: now also J1.202 (P202)
- net SPARE_P203: now also J1.203 (P203)
- net SPARE_P204: now also J1.204 (P204)
- net SPARE_P205: now also J1.205 (P205)
- net SPARE_P206: now also J1.206 (P206)
- net SPARE_P207: now also J1.207 (P207)
- net SPARE_P208: now also J1.208 (P208)
- net SPARE_P209: now also J1.209 (P209)
- net SPARE_P210: now also J1.210 (P210)
- net SPARE_P211: now also J1.211 (P211)
- net SPARE_P212: now also J1.212 (P212)
- net SPARE_P213: now also J1.213 (P213)
- net SPARE_P214: now also J1.214 (P214)
- net SPARE_P215: now also J1.215 (P215)
- net SPARE_P216: now also J1.216 (P216)
- net SPARE_P217: now also J1.217 (P217)
- net SPARE_P218: now also J1.218 (P218)
- net SPARE_P219: now also J1.219 (P219)
- net SPARE_P220: now also J1.220 (P220)
- net SPARE_P221: now also J1.221 (P221)
- net SPARE_P222: now also J1.222 (P222)
- net SPARE_P223: now also J1.223 (P223)
- net SPARE_P224: now also J1.224 (P224)
- net SPARE_P225: now also J1.225 (P225)
- net SPARE_P226: now also J1.226 (P226)
- net SPARE_P227: now also J1.227 (P227)
- net SPARE_P228: now also J1.228 (P228)
- net SPARE_P229: now also J1.229 (P229)
- net SPARE_P230: now also J1.230 (P230)
- net SPARE_P231: now also J1.231 (P231)
- net SPARE_P232: now also J1.232 (P232)
- net SPARE_P233: now also J1.233 (P233)
- net SPARE_P234: now also J1.234 (P234)
- net SPARE_P235: now also J1.235 (P235)
- net SPARE_P236: now also J1.236 (P236)
- net SPARE_P237: now also J1.237 (P237)
- net SPARE_P238: now also J1.238 (P238)
- net SPARE_P239: now also J1.239 (P239)
- net SPARE_P240: now also J1.240 (P240)
- net SSI0_CE0: now also J1.127 (P127)
- net SSI0_CE1: now also J1.128 (P128)
- net SSI0_CLK: now also J1.124 (P124)
- net SSI0_DR: now also J1.126 (P126)
- net SSI0_DT: now also J1.125 (P125)
- net SSI0_GPC: now also J1.129 (P129)
- net SSI1_CE0: now also J1.134 (P134)
- net SSI1_CLK: now also J1.131 (P131)
- net SSI1_DR: now also J1.133 (P133)
- net SSI1_DT: now also J1.132 (P132)
- net UART0_CTS: now also J1.100 (P100)
- net UART0_RTS: now also J1.101 (P101)
- net UART0_RXD: now also J1.98 (P98)
- net UART0_TXD: now also J1.99 (P99)
- net UART1_RX: now also J1.42 (P42)
- net UART1_TX: now also J1.43 (P43)
- net UART2_CTS: now also J1.105 (P105)
- net UART2_RTS: now also J1.106 (P106)
- net UART2_RXD: now also J1.103 (P103)
- net UART2_TXD: now also J1.104 (P104)
- net UART3_CTS: now also J1.110 (P110)
- net UART3_RTS: now also J1.111 (P111)
- net UART3_RXD: now also J1.108 (P108)
- net UART3_TXD: now also J1.109 (P109)
- net USBA_HOST_DM: now also J1.21 (P21)
- net USBA_HOST_DP: now also J1.20 (P20)
- net VCORE: now also J1.1 (P1), J1.2 (P2), J1.3 (P3), J1.4 (P4)
- net VCORE_SNS: now also J1.23 (P23)
- net VDDR: now also J1.10 (P10), J1.9 (P9)
- new net MSC0_CD: J4.10 (DET_A), R43.2

Commit message: Carrier: S5 pull-ups, unused-pin test-pad breakouts, value-only silk
- Add R44-R49 (100k) pull-ups/pull-downs for the BMC<->SoC link, SFC_IO2/IO3 and NOR CE
- Break out unused U15 P11-P17, U8 SPIIO7/MTMS/console UART and U12 spare VBUS to 1.0mm test pads
- Tie J4 SHIELD and J6 G to GND; no-connect the remaining unused pins (ERC pin_not_connected 30 -> 0)
- Silkscreen: show values/part names instead of references for R/C/U/L/D/Q/SW/JP (J refs kept)
- Refill zones; remove stray no-net track segments
- Interposer: SFC shared-bus pinout/schematic updates
Parts:
- added unit 2 of J1
- added unit 3 of J1
- added unit 4 of J1
- added unit 5 of J1
- added unit 6 of J1
- added R44, R45, R46, R47, R48, R49: 100k, Resistor_SMD:R_0402_1005Metric, symbol Device:R
- added TP1, TP10, TP11, TP12, TP13, TP2, TP3, TP4, TP5, TP6, TP7, TP8, TP9: TestPoint, TestPoint:TestPoint_Pad_D1.0mm, symbol Connector:TestPoint
- J1: footprint (none) -> teacup-carrier:DDR4288S0511H_UDIMM288
Connections:
- net +3V3: now also R44.1, R46.1, R47.1, R48.1, R49.1
- net EN_CS_U4: now also R44.2
- net EN_CS_U5: now also R45.1
- net ESP32_CONSOLE_RX: now also TP10.1
- net ESP32_CONSOLE_TX: now also TP11.1
- net GMAC0_MDCK: now also J1.88 (P88); no longer J1.88 (P88)
- net GMAC0_MDIO: now also J1.87 (P87); no longer J1.87 (P87)
- net GMAC0_PHYCLK: now also J1.90 (P90); no longer J1.90 (P90)
- net GMAC0_RXD0: now also J1.95 (P95); no longer J1.95 (P95)
- net GMAC0_RXD1: now also J1.96 (P96); no longer J1.96 (P96)
- net GMAC0_RXDV: now also J1.94 (P94); no longer J1.94 (P94)
- net GMAC0_TXCLK: now also J1.89 (P89); no longer J1.89 (P89)
- net GMAC0_TXD0: now also J1.92 (P92); no longer J1.92 (P92)
- net GMAC0_TXD1: now also J1.93 (P93); no longer J1.93 (P93)
- net GMAC0_TXEN: now also J1.91 (P91); no longer J1.91 (P91)
- net GMAC1_MDCK: now also J1.114 (P114); no longer J1.114 (P114)
- net GMAC1_MDIO: now also J1.113 (P113); no longer J1.113 (P113)
- net GMAC1_PHYCLK: now also J1.116 (P116); no longer J1.116 (P116)
- net GMAC1_RXD0: now also J1.121 (P121); no longer J1.121 (P121)
- net GMAC1_RXD1: now also J1.122 (P122); no longer J1.122 (P122)
- net GMAC1_RXDV: now also J1.120 (P120); no longer J1.120 (P120)
- net GMAC1_TXCLK: now also J1.115 (P115); no longer J1.115 (P115)
- net GMAC1_TXD0: now also J1.118 (P118); no longer J1.118 (P118)
- net GMAC1_TXD1: now also J1.119 (P119); no longer J1.119 (P119)
- net GMAC1_TXEN: now also J1.117 (P117); no longer J1.117 (P117)
- net GND: now also J4.11 (SHIELD), J6.G, J1.102 (P102), J1.107 (P107), J1.112 (P112), J1.123 (P123), J1.130 (P130), J1.135 (P135), J1.144 (P144), J1.145 (P145), J1.147 (P147), J1.152 (P152), J1.169 (P169), J1.170 (P170), J1.171 (P171), J1.172 (P172), J1.49 (P49), J1.51 (P51), J1.57 (P57), J1.58 (P58), J1.59 (P59), J1.63 (P63), J1.66 (P66), J1.69 (P69), J1.72 (P72), J1.76 (P76), J1.79 (P79), J1.82 (P82), J1.85 (P85), J1.86 (P86), J1.97 (P97), R45.2; no longer J1.102 (P102), J1.107 (P107), J1.112 (P112), J1.123 (P123), J1.130 (P130), J1.135 (P135), J1.144 (P144), J1.145 (P145), J1.147 (P147), J1.152 (P152), J1.169 (P169), J1.170 (P170), J1.171 (P171), J1.172 (P172), J1.49 (P49), J1.51 (P51), J1.57 (P57), J1.58 (P58), J1.59 (P59), J1.63 (P63), J1.66 (P66), J1.69 (P69), J1.72 (P72), J1.76 (P76), J1.79 (P79), J1.82 (P82), J1.85 (P85), J1.86 (P86), J1.97 (P97)
- net GPIO0: now also J1.153 (P153); no longer J1.153 (P153)
- net GPIO1: now also J1.154 (P154); no longer J1.154 (P154)
- net GPIO10: now also J1.163 (P163); no longer J1.163 (P163)
- net GPIO11: now also J1.164 (P164); no longer J1.164 (P164)
- net GPIO12: now also J1.165 (P165); no longer J1.165 (P165)
- net GPIO13: now also J1.166 (P166); no longer J1.166 (P166)
- net GPIO14: now also J1.167 (P167); no longer J1.167 (P167)
- net GPIO15: now also J1.168 (P168); no longer J1.168 (P168)
- net GPIO2: now also J1.155 (P155); no longer J1.155 (P155)
- net GPIO3: now also J1.156 (P156); no longer J1.156 (P156)
- net GPIO4: now also J1.157 (P157); no longer J1.157 (P157)
- net GPIO5: now also J1.158 (P158); no longer J1.158 (P158)
- net GPIO6: now also J1.159 (P159); no longer J1.159 (P159)
- net GPIO7: now also J1.160 (P160); no longer J1.160 (P160)
- net GPIO8: now also J1.161 (P161); no longer J1.161 (P161)
- net GPIO9: now also J1.162 (P162); no longer J1.162 (P162)
- net MIPI0_CLKN: now also J1.65 (P65); no longer J1.65 (P65)
- net MIPI0_CLKP: now also J1.64 (P64); no longer J1.64 (P64)
- net MIPI0_D0N: now also J1.71 (P71); no longer J1.71 (P71)
- net MIPI0_D0P: now also J1.70 (P70); no longer J1.70 (P70)
- net MIPI0_D1N: now also J1.68 (P68); no longer J1.68 (P68)
- net MIPI0_D1P: now also J1.67 (P67); no longer J1.67 (P67)
- net MIPI0_GPIO: now also J1.62 (P62); no longer J1.62 (P62)
- net MIPI0_SCCB_SCL: now also J1.61 (P61); no longer J1.61 (P61)
- net MIPI0_SCCB_SDA: now also J1.60 (P60); no longer J1.60 (P60)
- net MIPI1_CLKN: now also J1.78 (P78); no longer J1.78 (P78)
- net MIPI1_CLKP: now also J1.77 (P77); no longer J1.77 (P77)
- net MIPI1_D0N: now also J1.84 (P84); no longer J1.84 (P84)
- net MIPI1_D0P: now also J1.83 (P83); no longer J1.83 (P83)
- net MIPI1_D1N: now also J1.81 (P81); no longer J1.81 (P81)
- net MIPI1_D1P: now also J1.80 (P80); no longer J1.80 (P80)
- net MIPI1_GPIO: now also J1.75 (P75); no longer J1.75 (P75)
- net MIPI1_SCCB_SCL: now also J1.74 (P74); no longer J1.74 (P74)
- net MIPI1_SCCB_SDA: now also J1.73 (P73); no longer J1.73 (P73)
- net MSC0_CLK: now also J1.53 (P53); no longer J1.53 (P53)
- net MSC0_CMD: now also J1.54 (P54); no longer J1.54 (P54)
- net MSC0_D0: now also J1.52 (P52); no longer J1.52 (P52)
- net MSC0_D1: now also J1.50 (P50); no longer J1.50 (P50)
- net MSC0_D2: now also J1.56 (P56); no longer J1.56 (P56)
- net MSC0_D3_CD: now also J1.55 (P55); no longer J1.55 (P55)
- net MSC1_CLK: now also J1.283 (P283); no longer J1.283 (P283)
- net MSC1_CMD: now also J1.284 (P284); no longer J1.284 (P284)
- net MSC1_D0: now also J1.285 (P285); no longer J1.285 (P285)
- net MSC1_D1: now also J1.286 (P286); no longer J1.286 (P286)
- net MSC1_D2: now also J1.287 (P287); no longer J1.287 (P287)
- net MSC1_D3_CD: now also J1.288 (P288); no longer J1.288 (P288)
- net NOR_U4_CE: now also R48.2
- net NOR_U5_CE: now also R49.2
- net PWM0: now also J1.136 (P136); no longer J1.136 (P136)
- net PWM1: now also J1.137 (P137); no longer J1.137 (P137)
- net PWM2: now also J1.138 (P138); no longer J1.138 (P138)
- net PWM3: now also J1.139 (P139); no longer J1.139 (P139)
- net PWM4: now also J1.140 (P140); no longer J1.140 (P140)
- net PWM5: now also J1.141 (P141); no longer J1.141 (P141)
- net PWM6: now also J1.142 (P142); no longer J1.142 (P142)
- net PWM7: now also J1.143 (P143); no longer J1.143 (P143)
- net SAR_AUX0: now also J1.146 (P146); no longer J1.146 (P146)
- net SFC_IO2: now also R46.2
- net SFC_IO3: now also R47.2
- net SMB0_SCK: now also J1.149 (P149); no longer J1.149 (P149)
- net SMB0_SDA: now also J1.148 (P148); no longer J1.148 (P148)
- net SMB1_SCK: now also J1.151 (P151); no longer J1.151 (P151)
- net SMB1_SDA: now also J1.150 (P150); no longer J1.150 (P150)
- net SPARE_P173: now also J1.173 (P173); no longer J1.173 (P173)
- net SPARE_P174: now also J1.174 (P174); no longer J1.174 (P174)
- net SPARE_P175: now also J1.175 (P175); no longer J1.175 (P175)
- net SPARE_P176: now also J1.176 (P176); no longer J1.176 (P176)
- net SPARE_P177: now also J1.177 (P177); no longer J1.177 (P177)
- net SPARE_P178: now also J1.178 (P178); no longer J1.178 (P178)
- net SPARE_P179: now also J1.179 (P179); no longer J1.179 (P179)
- net SPARE_P180: now also J1.180 (P180); no longer J1.180 (P180)
- net SPARE_P181: now also J1.181 (P181); no longer J1.181 (P181)
- net SPARE_P182: now also J1.182 (P182); no longer J1.182 (P182)
- net SPARE_P183: now also J1.183 (P183); no longer J1.183 (P183)
- net SPARE_P184: now also J1.184 (P184); no longer J1.184 (P184)
- net SPARE_P185: now also J1.185 (P185); no longer J1.185 (P185)
- net SPARE_P186: now also J1.186 (P186); no longer J1.186 (P186)
- net SPARE_P187: now also J1.187 (P187); no longer J1.187 (P187)
- net SPARE_P188: now also J1.188 (P188); no longer J1.188 (P188)
- net SPARE_P189: now also J1.189 (P189); no longer J1.189 (P189)
- net SPARE_P190: now also J1.190 (P190); no longer J1.190 (P190)
- net SPARE_P191: now also J1.191 (P191); no longer J1.191 (P191)
- net SPARE_P192: now also J1.192 (P192); no longer J1.192 (P192)
- net SPARE_P193: now also J1.193 (P193); no longer J1.193 (P193)
- net SPARE_P194: now also J1.194 (P194); no longer J1.194 (P194)
- net SPARE_P195: now also J1.195 (P195); no longer J1.195 (P195)
- net SPARE_P196: now also J1.196 (P196); no longer J1.196 (P196)
- net SPARE_P197: now also J1.197 (P197); no longer J1.197 (P197)
- net SPARE_P198: now also J1.198 (P198); no longer J1.198 (P198)
- net SPARE_P199: now also J1.199 (P199); no longer J1.199 (P199)
- net SPARE_P200: now also J1.200 (P200); no longer J1.200 (P200)
- net SPARE_P201: now also J1.201 (P201); no longer J1.201 (P201)
- net SPARE_P202: now also J1.202 (P202); no longer J1.202 (P202)
- net SPARE_P203: now also J1.203 (P203); no longer J1.203 (P203)
- net SPARE_P204: now also J1.204 (P204); no longer J1.204 (P204)
- net SPARE_P205: now also J1.205 (P205); no longer J1.205 (P205)
- net SPARE_P206: now also J1.206 (P206); no longer J1.206 (P206)
- net SPARE_P207: now also J1.207 (P207); no longer J1.207 (P207)
- net SPARE_P208: now also J1.208 (P208); no longer J1.208 (P208)
- net SPARE_P209: now also J1.209 (P209); no longer J1.209 (P209)
- net SPARE_P210: now also J1.210 (P210); no longer J1.210 (P210)
- net SPARE_P211: now also J1.211 (P211); no longer J1.211 (P211)
- net SPARE_P212: now also J1.212 (P212); no longer J1.212 (P212)
- net SPARE_P213: now also J1.213 (P213); no longer J1.213 (P213)
- net SPARE_P214: now also J1.214 (P214); no longer J1.214 (P214)
- net SPARE_P215: now also J1.215 (P215); no longer J1.215 (P215)
- net SPARE_P216: now also J1.216 (P216); no longer J1.216 (P216)
- net SPARE_P217: now also J1.217 (P217); no longer J1.217 (P217)
- net SPARE_P218: now also J1.218 (P218); no longer J1.218 (P218)
- net SPARE_P219: now also J1.219 (P219); no longer J1.219 (P219)
- net SPARE_P220: now also J1.220 (P220); no longer J1.220 (P220)
- net SPARE_P221: now also J1.221 (P221); no longer J1.221 (P221)
- net SPARE_P222: now also J1.222 (P222); no longer J1.222 (P222)
- net SPARE_P223: now also J1.223 (P223); no longer J1.223 (P223)
- net SPARE_P224: now also J1.224 (P224); no longer J1.224 (P224)
- net SPARE_P225: now also J1.225 (P225); no longer J1.225 (P225)
- net SPARE_P226: now also J1.226 (P226); no longer J1.226 (P226)
- net SPARE_P227: now also J1.227 (P227); no longer J1.227 (P227)
- net SPARE_P228: now also J1.228 (P228); no longer J1.228 (P228)
- net SPARE_P229: now also J1.229 (P229); no longer J1.229 (P229)
- net SPARE_P230: now also J1.230 (P230); no longer J1.230 (P230)
- net SPARE_P231: now also J1.231 (P231); no longer J1.231 (P231)
- net SPARE_P232: now also J1.232 (P232); no longer J1.232 (P232)
- net SPARE_P233: now also J1.233 (P233); no longer J1.233 (P233)
- net SPARE_P234: now also J1.234 (P234); no longer J1.234 (P234)
- net SPARE_P235: now also J1.235 (P235); no longer J1.235 (P235)
- net SPARE_P236: now also J1.236 (P236); no longer J1.236 (P236)
- net SPARE_P237: now also J1.237 (P237); no longer J1.237 (P237)
- net SPARE_P238: now also J1.238 (P238); no longer J1.238 (P238)
- net SPARE_P239: now also J1.239 (P239); no longer J1.239 (P239)
- net SPARE_P240: now also J1.240 (P240); no longer J1.240 (P240)
- net SPARE_P241: now also J1.241 (P241); no longer J1.241 (P241)
- net SPARE_P242: now also J1.242 (P242); no longer J1.242 (P242)
- net SPARE_P243: now also J1.243 (P243); no longer J1.243 (P243)
- net SPARE_P244: now also J1.244 (P244); no longer J1.244 (P244)
- net SPARE_P245: now also J1.245 (P245); no longer J1.245 (P245)
- net SPARE_P246: now also J1.246 (P246); no longer J1.246 (P246)
- net SPARE_P247: now also J1.247 (P247); no longer J1.247 (P247)
- net SPARE_P248: now also J1.248 (P248); no longer J1.248 (P248)
- net SPARE_P249: now also J1.249 (P249); no longer J1.249 (P249)
- net SPARE_P250: now also J1.250 (P250); no longer J1.250 (P250)
- net SPARE_P251: now also J1.251 (P251); no longer J1.251 (P251)
- net SPARE_P252: now also J1.252 (P252); no longer J1.252 (P252)
- net SPARE_P253: now also J1.253 (P253); no longer J1.253 (P253)
- net SPARE_P254: now also J1.254 (P254); no longer J1.254 (P254)
- net SPARE_P255: now also J1.255 (P255); no longer J1.255 (P255)
- net SPARE_P256: now also J1.256 (P256); no longer J1.256 (P256)
- net SPARE_P257: now also J1.257 (P257); no longer J1.257 (P257)
- net SPARE_P258: now also J1.258 (P258); no longer J1.258 (P258)
- net SPARE_P259: now also J1.259 (P259); no longer J1.259 (P259)
- net SPARE_P260: now also J1.260 (P260); no longer J1.260 (P260)
- net SPARE_P261: now also J1.261 (P261); no longer J1.261 (P261)
- net SPARE_P262: now also J1.262 (P262); no longer J1.262 (P262)
- net SPARE_P263: now also J1.263 (P263); no longer J1.263 (P263)
- net SPARE_P264: now also J1.264 (P264); no longer J1.264 (P264)
- net SPARE_P265: now also J1.265 (P265); no longer J1.265 (P265)
- net SPARE_P266: now also J1.266 (P266); no longer J1.266 (P266)
- net SPARE_P267: now also J1.267 (P267); no longer J1.267 (P267)
- net SPARE_P268: now also J1.268 (P268); no longer J1.268 (P268)
- net SPARE_P269: now also J1.269 (P269); no longer J1.269 (P269)
- net SPARE_P270: now also J1.270 (P270); no longer J1.270 (P270)
- net SPARE_P271: now also J1.271 (P271); no longer J1.271 (P271)
- net SPARE_P272: now also J1.272 (P272); no longer J1.272 (P272)
- net SPARE_P273: now also J1.273 (P273); no longer J1.273 (P273)
- net SPARE_P274: now also J1.274 (P274); no longer J1.274 (P274)
- net SPARE_P275: now also J1.275 (P275); no longer J1.275 (P275)
- net SPARE_P276: now also J1.276 (P276); no longer J1.276 (P276)
- net SPARE_P277: now also J1.277 (P277); no longer J1.277 (P277)
- net SPARE_P278: now also J1.278 (P278); no longer J1.278 (P278)
- net SPARE_P279: now also J1.279 (P279); no longer J1.279 (P279)
- net SPARE_P280: now also J1.280 (P280); no longer J1.280 (P280)
- net SPARE_P281: now also J1.281 (P281); no longer J1.281 (P281)
- net SPARE_P282: now also J1.282 (P282); no longer J1.282 (P282)
- net SSI0_CE0: now also J1.127 (P127); no longer J1.127 (P127)
- net SSI0_CE1: now also J1.128 (P128); no longer J1.128 (P128)
- net SSI0_CLK: now also J1.124 (P124); no longer J1.124 (P124)
- net SSI0_DR: now also J1.126 (P126); no longer J1.126 (P126)
- net SSI0_DT: now also J1.125 (P125); no longer J1.125 (P125)
- net SSI0_GPC: now also J1.129 (P129); no longer J1.129 (P129)
- net SSI1_CE0: now also J1.134 (P134); no longer J1.134 (P134)
- net SSI1_CLK: now also J1.131 (P131); no longer J1.131 (P131)
- net SSI1_DR: now also J1.133 (P133); no longer J1.133 (P133)
- net SSI1_DT: now also J1.132 (P132); no longer J1.132 (P132)
- net UART0_CTS: now also J1.100 (P100); no longer J1.100 (P100)
- net UART0_RTS: now also J1.101 (P101); no longer J1.101 (P101)
- net UART0_RXD: now also J1.98 (P98); no longer J1.98 (P98)
- net UART0_TXD: now also J1.99 (P99); no longer J1.99 (P99)
- net UART2_CTS: now also J1.105 (P105); no longer J1.105 (P105)
- net UART2_RTS: now also J1.106 (P106); no longer J1.106 (P106)
- net UART2_RXD: now also J1.103 (P103); no longer J1.103 (P103)
- net UART2_TXD: now also J1.104 (P104); no longer J1.104 (P104)
- net UART3_CTS: now also J1.110 (P110); no longer J1.110 (P110)
- net UART3_RTS: now also J1.111 (P111); no longer J1.111 (P111)
- net UART3_RXD: now also J1.108 (P108); no longer J1.108 (P108)
- net UART3_TXD: now also J1.109 (P109); no longer J1.109 (P109)
- net USB2_VBUS_OUT: now also TP12.1
- net USB3_VBUS_OUT: now also TP13.1
- net at U8.29 (SPIIO7): now also TP8.1
- net at U8.35 (MTMS): now also TP9.1
- net at U15.14 (P11): now also TP1.1
- net at U15.15 (P12): now also TP2.1
- net at U15.16 (P13): now also TP3.1
- net at U15.17 (P14): now also TP4.1
- net at U15.18 (P15): now also TP5.1
- net at U15.19 (P16): now also TP6.1
- net at U15.20 (P17): now also TP7.1
- no-connect marks 0 -> 19
Other:
- moved on the sheet: C21, C22, R41, R42, R8, R9, U10, U9

Commit message: Restore MPN/Manufacturer fields lost in upstream merge resolution
The upstream/main merge resolved the carrier + T31 interposer .kicad_sch
conflicts with --ours, which dropped upstream's MPN backfill (PR #17). Re-add
MPN/Manufacturer for the 28 carrier parts and interposer IC1.
Parts:
- D1, D2: MPN (none) -> PMEG2010ER; Manufacturer (none) -> Nexperia
- J1: MPN (none) -> AH58893-T9B10-3F
- J2, J9: MPN (none) -> TYPE-C-31-M-12; Manufacturer (none) -> Hroparts Elec
- J3: MPN (none) -> 292303-7; Manufacturer (none) -> TE Connectivity
- J4: MPN (none) -> DM3D-SF; Manufacturer (none) -> Hirose Electric
- J5: MPN (none) -> 694106301002; Manufacturer (none) -> Wurth Elektronik
- J7, J8: MPN (none) -> SFW15R-2STE1LF; Manufacturer (none) -> JAE Electronics
- Q1, Q2: MPN (none) -> AO3401A; Manufacturer (none) -> Alpha & Omega Semiconductor
- SW1, SW2: MPN (none) -> SSSS711403
- U1: MPN (none) -> AP62600SJ-7; Manufacturer (none) -> Diodes Incorporated
- U10, U9: MPN (none) -> TS5A3166; Manufacturer (none) -> Texas Instruments
- U12: MPN (none) -> TPS2053BDR; Manufacturer (none) -> Texas Instruments
- U13: MPN (none) -> W25Q32JVSS; Manufacturer (none) -> Winbond Electronics
- U14: MPN (none) -> TPS22990DMLR; Manufacturer (none) -> Texas Instruments
- U15: MPN (none) -> TCA9555PWR; Manufacturer (none) -> Texas Instruments
- U2, U7: MPN (none) -> AP62300WU-7; Manufacturer (none) -> Diodes Incorporated
- U3: MPN (none) -> MCP4661-104E/ST; Manufacturer (none) -> Microchip Technology
- U6: MPN (none) -> AZ1117CH-1.8TRG1
- U8: MPN (none) -> ESP32-S3-WROOM-1-N16R2; Manufacturer (none) -> Espressif Systems
