File: hw/teacup-carrier.kicad_pcb (KiCad board)
At the start: 4 copper layers, 257 x 117.5 mm, 137 parts, among them J1 AH58893-T9B10-3F, J2 TYPE-C-31-M-12, J20 HDR_J20, J21 HDR_J21, J22 HDR_J22, J23 HDR_J23, J24 HDR_J24, J25 HDR_J25, J26 HDR_J26, J27 HDR_J27, J28 HDR_J28, J29 HDR_J29, J3 TE_292303-7, J30 HDR_J30, J31 HDR_J31, J32 HDR_J32, J33 HDR_J33, J34 HDR_J34, J35 HDR_J35, J36 HDR_J36, J37 HDR_J37, J38 AMP_MIC_TAP, J4 Hirose_DM3D-SF, J5 Wuerth_694106301002, J6 AudioJack4_Ground, J7 SFW15R-2STE1LF, J8 SFW15R-2STE1LF, J9 TYPE-C-31-M-12, Q1 AO3401A, Q2 AO3401A, SW1 SSSS711403, SW2 SSSS711403, U1 AP62600SJ-7, U10 TS5A3166, U11 DIP-8 Socket, U12 TPS2053BDR, U13 W25Q32JVSS, U14 TPS22990DMLR, U15 TCA9555PWR, U2 AP62300WU-7, U3 MCP4661-104E_ST, U4 TPS22990DMLR, U5 AZ1117CH-3.3TRG1, U6 AZ1117CH-1.8TRG1, U7 AP62300WU-7, U8 ESP32-S3-WROOM-1-N16R2, U9 TS5A3166

Commit message: Add net class clearance rule and continue manual PCB routing
Set Default net class clearance to 0.15mm, matching TeaCup 3.3's DRC
rules. PCB routing continues from manual work in KiCad; DRC still has
open items (clearance/solder-mask-bridge) to clean up in a follow-up.
Parts:
- moved C12 75.9 mm to (87.8, 87.5)
- moved C14 75.9 mm to (91.7, 100.3)
- moved C15 75.9 mm to (91.5, 103.6)
- moved C19 75.9 mm to (91.6, 87.4)
- moved C20 75.9 mm to (91.4, 91.5)
- moved U5 75.9 mm to (98.2, 101.8)
- moved U6 75.9 mm to (98.1, 89.5)
- moved C29 40.5 mm to (68.7, 120.2)
- moved R14 33.8 mm to (65.3, 124.3), turned to 90 degrees
- moved J37 15.2 mm to (265.3, 83.1), turned to -90 degrees
- moved R7 13.7 mm to (51.4, 79.2), turned to 90 degrees
- moved U13 10.4 mm to (130.9, 91.2)
- moved U10 10.4 mm to (115.2, 104.2)
- moved C24 10.4 mm to (140.2, 90.6)
- moved U11 10.4 mm to (115.9, 87.3)
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Routing:
- net SSI0_GPC: track 0.00 -> 87.3 mm
- net SSI0_CE0: track 0.00 -> 85.6 mm
- net SSI0_DT: track 0.00 -> 84.5 mm
- net SSI0_CE1: track 0.00 -> 83.4 mm
- net SSI0_DR: track 0.00 -> 81.8 mm
- net SSI0_CLK: track 0.00 -> 80.9 mm
- net SSI1_CE0: track 0.00 -> 78.1 mm
- net GMAC1_MDCK: track 0.00 -> 77.8 mm
- net GMAC1_PHYCLK: track 0.00 -> 77.8 mm
- net GMAC1_TXD0: track 0.00 -> 77.7 mm
- net GMAC1_RXDV: track 0.00 -> 77.6 mm
- net GMAC1_RXD1: track 0.00 -> 77.5 mm
- net SSI1_DR: track 0.00 -> 76.7 mm
- net GMAC1_MDIO: track 0.00 -> 74.8 mm
- net SSI1_DT: track 0.00 -> 74.8 mm
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