File: hw/teacup-carrier.kicad_pcb (KiCad board)
At the start: 4 copper layers, 257 x 117.5 mm, 137 parts, among them J1 AH58893-T9B10-3F, J2 TYPE-C-31-M-12, J20 HDR_J20, J21 HDR_J21, J22 HDR_J22, J23 HDR_J23, J24 HDR_J24, J25 HDR_J25, J26 HDR_J26, J27 HDR_J27, J28 HDR_J28, J29 HDR_J29, J3 TE_292303-7, J30 HDR_J30, J31 HDR_J31, J32 HDR_J32, J33 HDR_J33, J34 HDR_J34, J35 HDR_J35, J36 HDR_J36, J37 HDR_J37, J38 AMP_MIC_TAP, J4 Hirose_DM3D-SF, J5 Wuerth_694106301002, J6 AudioJack4_Ground, J7 SFW15R-2STE1LF, J8 SFW15R-2STE1LF, J9 TYPE-C-31-M-12, Q1 AO3401A, Q2 AO3401A, SW1 SSSS711403, SW2 SSSS711403, U1 AP62600SJ-7, U10 TS5A3166, U11 DIP-8 Socket, U12 TPS2053BDR, U13 W25Q32JVSS, U14 TPS22990DMLR, U15 TCA9555PWR, U2 AP62300WU-7, U3 MCP4661-104E_ST, U4 TPS22990DMLR, U5 AZ1117CH-3.3TRG1, U6 AZ1117CH-1.8TRG1, U7 AP62300WU-7, U8 ESP32-S3-WROOM-1-N16R2, U9 TS5A3166

Commit message: Carrier: S5 pull-ups, unused-pin test-pad breakouts, value-only silk
- Add R44-R49 (100k) pull-ups/pull-downs for the BMC<->SoC link, SFC_IO2/IO3 and NOR CE
- Break out unused U15 P11-P17, U8 SPIIO7/MTMS/console UART and U12 spare VBUS to 1.0mm test pads
- Tie J4 SHIELD and J6 G to GND; no-connect the remaining unused pins (ERC pin_not_connected 30 -> 0)
- Silkscreen: show values/part names instead of references for R/C/U/L/D/Q/SW/JP (J refs kept)
- Refill zones; remove stray no-net track segments
- Interposer: SFC shared-bus pinout/schematic updates
Parts:
- added C20: 10uF, Capacitor_SMD:C_0805_2012Metric, F.Cu at (90.9, 75.2)
- added R44: 100k, Resistor_SMD:R_0402_1005Metric, F.Cu at (109.6, 91.6)
- added R45: 100k, Resistor_SMD:R_0402_1005Metric, F.Cu at (107.3, 98.3)
- added R46: 100k, Resistor_SMD:R_0402_1005Metric, F.Cu at (144.6, 123.1)
- added R47: 100k, Resistor_SMD:R_0402_1005Metric, F.Cu at (157.9, 121.0)
- added R48: 100k, Resistor_SMD:R_0402_1005Metric, F.Cu at (144.5, 118.2)
- added R49: 100k, Resistor_SMD:R_0402_1005Metric, F.Cu at (144.4, 126.5)
- added TP1: TestPoint, TestPoint:TestPoint_Pad_D1.0mm, F.Cu at (103.2, 94.3)
- added TP10: TestPoint, TestPoint:TestPoint_Pad_D1.0mm, F.Cu at (111.2, 99.5)
- added TP11: TestPoint, TestPoint:TestPoint_Pad_D1.0mm, F.Cu at (112.5, 101.4)
- added TP12: TestPoint, TestPoint:TestPoint_Pad_D1.0mm, F.Cu at (104.2, 101.9)
- added TP13: TestPoint, TestPoint:TestPoint_Pad_D1.0mm, F.Cu at (104.2, 106.0)
- added TP2: TestPoint, TestPoint:TestPoint_Pad_D1.0mm, F.Cu at (105.4, 94.3)
- added TP3: TestPoint, TestPoint:TestPoint_Pad_D1.0mm, F.Cu at (106.3, 92.5)
- added TP4: TestPoint, TestPoint:TestPoint_Pad_D1.0mm, F.Cu at (104.3, 92.6)
- added TP5: TestPoint, TestPoint:TestPoint_Pad_D1.0mm, F.Cu at (105.5, 90.7)
- added TP6: TestPoint, TestPoint:TestPoint_Pad_D1.0mm, F.Cu at (103.3, 90.9)
- added TP7: TestPoint, TestPoint:TestPoint_Pad_D1.0mm, F.Cu at (104.2, 89.1)
- added TP8: TestPoint, TestPoint:TestPoint_Pad_D1.0mm, F.Cu at (110.5, 84.5)
- added TP9: TestPoint, TestPoint:TestPoint_Pad_D1.0mm, F.Cu at (112.2, 97.1)
- U14, U4: footprint WSON-10_L3.0-W2.0-P0.50-BL-EP_TI_DML -> teacup-carrier:WSON-10_L3.0-W2.0-P0.50-BL-EP_TI_DML
- moved C25 6.12 mm to (104.0, 98.4)
Connections:
- U15 pad 14: unconnected-(U15-P11-Pad14) -> Net-(U15-P11)
- U15 pad 15: unconnected-(U15-P12-Pad15) -> Net-(U15-P12)
- U15 pad 16: unconnected-(U15-P13-Pad16) -> Net-(U15-P13)
- U15 pad 17: unconnected-(U15-P14-Pad17) -> Net-(U15-P14)
- U15 pad 18: unconnected-(U15-P15-Pad18) -> Net-(U15-P15)
- U15 pad 19: unconnected-(U15-P16-Pad19) -> Net-(U15-P16)
- U15 pad 20: unconnected-(U15-P17-Pad20) -> Net-(U15-P17)
- U8 pad 29: unconnected-(U8-SPIIO7-Pad29) -> Net-(U8-SPIIO7)
- U8 pad 35: unconnected-(U8-MTMS-Pad35) -> Net-(U8-MTMS)
Routing:
- net /ESP32_CONSOLE_TX: track 0.00 -> 8.85 mm
- net /ESP32_CONSOLE_RX: track 0.00 -> 8.82 mm
- net Net-(U8-MTMS): track 0.00 -> 7.58 mm
- net +3V3: track 55.6 -> 62.5 mm, vias 38 -> 42
- net GND: track 91.5 -> 97.4 mm, vias 46 -> 48
- net Net-(U15-P13): track 0.00 -> 5.56 mm
- net Net-(U8-SPIIO7): track 0.00 -> 4.96 mm
- net Net-(U15-P15): track 0.00 -> 4.79 mm
- net Net-(U15-P12): track 0.00 -> 4.54 mm
- net +1V8: track 0.85 -> 5.23 mm
- net Net-(U15-P17): track 0.00 -> 3.52 mm
- net USB3_VBUS_OUT: track 0.00 -> 3.39 mm
- net USB2_VBUS_OUT: track 0.00 -> 3.28 mm
- net Net-(U15-P14): track 0.00 -> 3.11 mm
- net EN_CS_U5: track 13.1 -> 15.6 mm
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