File: hw/sheets/bmc.kicad_sch (KiCad schematic)
At the start: 16 parts, among them SW1 SSSS711403, SW2 SSSS711403, U10 TS5A3166, U11 DIP-8 Socket, U12 TPS2053BDR, U13 W25Q32JVSS, U15 TCA9555PWR, U8 ESP32-S3-WROOM-1-N16R2, U9 TS5A3166

Commit message: Carrier board: fix 3 power/USB bugs, add missing passives, replace digipot-only VCORE/VDDR with jumper-selectable presets
Bugs found in a passive-component audit and fixed:
- U7 (+3V3 buck) EN was pulled from its own output (+3V3), a startup
  deadlock -- repointed to +5V_SW (its VIN), matching U1's pattern.
- U12 (TPS2053BDR USB power switch) IN1/IN2 were entirely unconnected --
  wired to +5V_SW.
- Neither I2C bus (I2C_PWR, I2C_ID) had a single pull-up resistor -- added
  4.7k to +3V3 on both, on the carrier side since it's always populated
  regardless of which interposer is seated.
- Added local decoupling at U3/U11/U13/U15 and bulk caps on every raw
  external rail (+5V_BMC, +5V_ALT, DCJACK_VBUS) before any regulator --
  none had local capacitance before.

VCORE/VDDR voltage-select jumpers (explicit design direction): U1/U2's FB
pins are now the common pole of a jumper bank rather than hard-wired to the
digipot wiper. 4 fixed presets for VCORE (0.8/0.9/1.0/1.1V) + 3 for VDDR
(1.35/1.5/1.8V), each a permanently-powered fixed divider, plus a
"computer" position that routes FB to the digipot exactly as before. This
makes VCORE/VDDR hardware-deterministic regardless of digipot NV memory or
EEPROM state -- solving not just first-power-up safety (the original JP1 +
mandatory bring-up checklist) but also the same gap reopening on every
interposer swap, which JP1 never covered. JP1 and the checklist are
removed; SW2's pole now ties directly to +5V_ALT.

Verified: 0 layout overlaps, full netlist diff shows only the intended 33
new components + JP1 removed + exactly 8 intentional pin rewires (nothing
else moved), ERC violation count/category breakdown consistent with the
established pattern (net +2, no new categories). Also switched the
verification toolchain to the actual installed KiCad (10.0.4 at
/opt/kicad10, matching the real GUI) after discovering the system
kicad-cli in PATH was a stray older 9.0.8.
Parts:
- removed JP1: PROVISIONED, Connector_PinHeader_2.54mm:PinHeader_1x02_P2.54mm_Vertical, symbol Connector_Generic:Conn_01x02
- added C24, C25, C26: 100nF, Capacitor_SMD:C_0402_1005Metric, symbol Device:C
- added R41, R42: 4.7k, Resistor_SMD:R_0402_1005Metric, symbol Device:R
Connections:
- net SW2_POLE is gone; now on net +5V_ALT: SW2.3
- net USB2_VBUS_IN is gone; now on net +5V_SW: U12.6 (IN2)
- net +3V3: now also C24.1, C25.1, C26.1, R41.1, R42.1
- net GND: now also C24.2, C25.2, C26.2
- net I2C_ID_SCL: now also R42.2
- net I2C_ID_SDA: now also R41.2
- net USB1_VBUS_IN renamed +5V_SW
