File: hw/sheets/power.kicad_sch (KiCad schematic)
At the start: 45 parts, among them U1 AP62600SJ-7, U14 TPS22990DMLR, U2 AP62300WU-7, U3 MCP4661-104E_ST, U4 TPS22990DMLR, U5 AZ1117CH-3.3TRG1, U6 AZ1117CH-1.8TRG1, U7 AP62300WU-7

Commit message: Carrier board: fix 3 power/USB bugs, add missing passives, replace digipot-only VCORE/VDDR with jumper-selectable presets
Bugs found in a passive-component audit and fixed:
- U7 (+3V3 buck) EN was pulled from its own output (+3V3), a startup
  deadlock -- repointed to +5V_SW (its VIN), matching U1's pattern.
- U12 (TPS2053BDR USB power switch) IN1/IN2 were entirely unconnected --
  wired to +5V_SW.
- Neither I2C bus (I2C_PWR, I2C_ID) had a single pull-up resistor -- added
  4.7k to +3V3 on both, on the carrier side since it's always populated
  regardless of which interposer is seated.
- Added local decoupling at U3/U11/U13/U15 and bulk caps on every raw
  external rail (+5V_BMC, +5V_ALT, DCJACK_VBUS) before any regulator --
  none had local capacitance before.

VCORE/VDDR voltage-select jumpers (explicit design direction): U1/U2's FB
pins are now the common pole of a jumper bank rather than hard-wired to the
digipot wiper. 4 fixed presets for VCORE (0.8/0.9/1.0/1.1V) + 3 for VDDR
(1.35/1.5/1.8V), each a permanently-powered fixed divider, plus a
"computer" position that routes FB to the digipot exactly as before. This
makes VCORE/VDDR hardware-deterministic regardless of digipot NV memory or
EEPROM state -- solving not just first-power-up safety (the original JP1 +
mandatory bring-up checklist) but also the same gap reopening on every
interposer swap, which JP1 never covered. JP1 and the checklist are
removed; SW2's pole now ties directly to +5V_ALT.

Verified: 0 layout overlaps, full netlist diff shows only the intended 33
new components + JP1 removed + exactly 8 intentional pin rewires (nothing
else moved), ERC violation count/category breakdown consistent with the
established pattern (net +2, no new categories). Also switched the
verification toolchain to the actual installed KiCad (10.0.4 at
/opt/kicad10, matching the real GUI) after discovering the system
kicad-cli in PATH was a stray older 9.0.8.
Parts:
- added JP10, JP6: COMPUTER, Connector_PinHeader_2.54mm:PinHeader_1x02_P2.54mm_Vertical, symbol Connector_Generic:Conn_01x02
- added JP2: 0.8V, Connector_PinHeader_2.54mm:PinHeader_1x02_P2.54mm_Vertical, symbol Connector_Generic:Conn_01x02
- added JP3: 0.9V, Connector_PinHeader_2.54mm:PinHeader_1x02_P2.54mm_Vertical, symbol Connector_Generic:Conn_01x02
- added JP4: 1.0V, Connector_PinHeader_2.54mm:PinHeader_1x02_P2.54mm_Vertical, symbol Connector_Generic:Conn_01x02
- added JP5: 1.1V, Connector_PinHeader_2.54mm:PinHeader_1x02_P2.54mm_Vertical, symbol Connector_Generic:Conn_01x02
- added JP7: 1.35V, Connector_PinHeader_2.54mm:PinHeader_1x02_P2.54mm_Vertical, symbol Connector_Generic:Conn_01x02
- added JP8: 1.5V, Connector_PinHeader_2.54mm:PinHeader_1x02_P2.54mm_Vertical, symbol Connector_Generic:Conn_01x02
- added JP9: 1.8V, Connector_PinHeader_2.54mm:PinHeader_1x02_P2.54mm_Vertical, symbol Connector_Generic:Conn_01x02
- added R25, R26: 4.7k, Resistor_SMD:R_0402_1005Metric, symbol Device:R
- added R27: 3.32k, Resistor_SMD:R_0402_1005Metric, symbol Device:R
- added R28, R30, R32, R34, R36, R38, R40: 10.0k, Resistor_SMD:R_0402_1005Metric, symbol Device:R
- added R29: 4.99k, Resistor_SMD:R_0402_1005Metric, symbol Device:R
- added R31: 6.65k, Resistor_SMD:R_0402_1005Metric, symbol Device:R
- added R33: 8.25k, Resistor_SMD:R_0402_1005Metric, symbol Device:R
- added R35: 6.81k, Resistor_SMD:R_0402_1005Metric, symbol Device:R
- added R37: 8.66k, Resistor_SMD:R_0402_1005Metric, symbol Device:R
- added R39: 12.4k, Resistor_SMD:R_0402_1005Metric, symbol Device:R
Connections:
- net +3V3: now also R25.1, R26.1; no longer R5.1
- net +5V_SW: now also R5.1
- net GND: now also R28.2, R30.2, R32.2, R34.2, R36.2, R38.2, R40.2
- net I2C_PWR_SCL: now also R26.2
- net I2C_PWR_SDA: now also R25.2
- net VCORE: now also R27.1, R29.1, R31.1, R33.1
- net VDDR: now also R35.1, R37.1, R39.1
- net VCORE_FB renamed VCORE_FB_DIGIPOT
- net VCORE_FB_DIGIPOT: now also JP6.2 (Pin_2); no longer U1.12 (FB)
- net VDDR_FB renamed VDDR_FB_DIGIPOT
- net VDDR_FB_DIGIPOT: now also JP10.2 (Pin_2); no longer U2.4 (FB)
- new net VCORE_FB_0V8: JP2.2 (Pin_2), R27.2, R28.1
- new net VCORE_FB_0V9: JP3.2 (Pin_2), R29.2, R30.1
- new net VCORE_FB_1V0: JP4.2 (Pin_2), R31.2, R32.1
- new net VCORE_FB_1V1: JP5.2 (Pin_2), R33.2, R34.1
- new net VCORE_FB_SEL: JP2.1 (Pin_1), JP3.1 (Pin_1), JP4.1 (Pin_1), JP5.1 (Pin_1), JP6.1 (Pin_1), U1.12 (FB)
- new net VDDR_FB_1V35: JP7.2 (Pin_2), R35.2, R36.1
- new net VDDR_FB_1V5: JP8.2 (Pin_2), R37.2, R38.1
- new net VDDR_FB_1V8: JP9.2 (Pin_2), R39.2, R40.1
- new net VDDR_FB_SEL: JP10.1 (Pin_1), JP7.1 (Pin_1), JP8.1 (Pin_1), JP9.1 (Pin_1), U2.4 (FB)
Other:
- note added: "VCORE VOLTAGE SELECT"
- note added: "VDDR VOLTAGE SELECT"
