File: hw/sheets/io.kicad_sch (KiCad schematic)
At the start: 18 parts, among them J2 TYPE-C-31-M-12, J3 TE_292303-7, J4 Hirose_DM3D-SF, J5 Wuerth_694106301002, J6 AudioJack4_Ground, J7 SFW15R-2STE1LF, J8 SFW15R-2STE1LF, J9 TYPE-C-31-M-12, Q1 AO3401A, Q2 AO3401A

Commit message: Carrier board: fix 3 power/USB bugs, add missing passives, replace digipot-only VCORE/VDDR with jumper-selectable presets
Bugs found in a passive-component audit and fixed:
- U7 (+3V3 buck) EN was pulled from its own output (+3V3), a startup
  deadlock -- repointed to +5V_SW (its VIN), matching U1's pattern.
- U12 (TPS2053BDR USB power switch) IN1/IN2 were entirely unconnected --
  wired to +5V_SW.
- Neither I2C bus (I2C_PWR, I2C_ID) had a single pull-up resistor -- added
  4.7k to +3V3 on both, on the carrier side since it's always populated
  regardless of which interposer is seated.
- Added local decoupling at U3/U11/U13/U15 and bulk caps on every raw
  external rail (+5V_BMC, +5V_ALT, DCJACK_VBUS) before any regulator --
  none had local capacitance before.

VCORE/VDDR voltage-select jumpers (explicit design direction): U1/U2's FB
pins are now the common pole of a jumper bank rather than hard-wired to the
digipot wiper. 4 fixed presets for VCORE (0.8/0.9/1.0/1.1V) + 3 for VDDR
(1.35/1.5/1.8V), each a permanently-powered fixed divider, plus a
"computer" position that routes FB to the digipot exactly as before. This
makes VCORE/VDDR hardware-deterministic regardless of digipot NV memory or
EEPROM state -- solving not just first-power-up safety (the original JP1 +
mandatory bring-up checklist) but also the same gap reopening on every
interposer swap, which JP1 never covered. JP1 and the checklist are
removed; SW2's pole now ties directly to +5V_ALT.

Verified: 0 layout overlaps, full netlist diff shows only the intended 33
new components + JP1 removed + exactly 8 intentional pin rewires (nothing
else moved), ERC violation count/category breakdown consistent with the
established pattern (net +2, no new categories). Also switched the
verification toolchain to the actual installed KiCad (10.0.4 at
/opt/kicad10, matching the real GUI) after discovering the system
kicad-cli in PATH was a stray older 9.0.8.
Parts:
- added C27, C28, C29: 10uF, Capacitor_SMD:C_0805_2012Metric, symbol Device:C
Connections:
- net +5V_ALT: now also C28.1
- net +5V_BMC: now also C27.1
- net DCJACK_VBUS: now also C29.1
- net GND: now also C27.2, C28.2, C29.2

Commit message: Fix Q1/Q2 pin mapping: Device:Q_PMOS -> Transistor_FET:AO3401A
Root cause of the PCB pass's 6 unassigned Q1/Q2 pins: Device:Q_PMOS is a
generic schematic-only placeholder whose pin NUMBERS are the letters
G/D/S themselves, never meant to auto-associate with a real footprint's
numeric pads. Switched to KiCad's dedicated AO3401A symbol (extends
TP0610T for its actual pin data, which schgen's simple loader doesn't
resolve automatically -- loaded TP0610T's body and cached/renamed it
under the AO3401A lib_id instead), which has real numeric pins matching
the manufacturer part and is already paired with the same SOT-23
footprint used here.

Pin assignment (1=G, 2=S, 3=D) verified against two independent sources
after KiCad's library and an initial visual read of AOS's own datasheet
diagram disagreed on the pin-2-vs-3 assignment -- confirmed via a second,
explicit numeric pin table from an independent source.

J6's remaining unassigned G pin is not a bug: checked against the
original single-SoC board's actual fabricated gerbers, which used this
identical symbol/footprint pair and never routed G to copper either (the
mounting holes are non-plated/NPTH, mechanical-only). Proven behavior.

Also: registered Transistor_FET in sym-lib-table (was missing, caused an
ERC library-not-found warning), taught gen_connections.py to follow
KiCad's (extends "Base") symbol inheritance so it can still read pins for
symbols like this one, and reverted an unrelated kicad-cli side effect
(silently strips the project's ERC-exclusions section on load -- known
issue from the previous PCB pass, not a real change).

Verified: netlist diff shows only Q1/Q2's pin identifiers changed
(letters -> matching numbers), nothing else moved. PCB rebuild: 1
remaining unassigned pin (J6/G, expected) vs 7 before. DRC: same 20
fine-pitch clearance violations as before, no new categories, zero
placement/courtyard regressions.
Parts:
- removed Q1, Q2: AO3401A, Package_TO_SOT_SMD:SOT-23, symbol Device:Q_PMOS
- added Q1, Q2: AO3401A, Package_TO_SOT_SMD:SOT-23, symbol Transistor_FET:AO3401A
Connections:
- net +5V_ALT: now also Q1.3 (D), Q2.3 (D)
- net ALTUSB_VBUS: now also Q2.2 (S)
- net DCJACK_VBUS: now also Q1.2 (S)
- net Q1_GATE: now also Q1.1 (G)
- net Q2_GATE: now also Q2.1 (G)
Changed lines of the file:
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@@
 		(property "Value" "GND" (at 82.55 135.89000000000001 0) (effects (font (size 1.27 1.27))))
 	)
-	(symbol (lib_id "Device:Q_PMOS") (at 114.3 165.1 0) (unit 1)
+	(symbol (lib_id "Transistor_FET:AO3401A") (at 114.3 165.1 0) (unit 1)
 		(property "Reference" "Q1" (at 104.14 161.29 0) (effects (font (size 1.27 1.27))))
 		(property "Value" "AO3401A" (at 104.14 168.91 0) (effects (font (size 1.27 1.27))))
@@
 		(property "Value" "GND" (at 114.3 193.04000000000002 0) (effects (font (size 1.27 1.27))))
 	)
-	(symbol (lib_id "Device:Q_PMOS") (at 133.35 165.1 0) (unit 1)
+	(symbol (lib_id "Transistor_FET:AO3401A") (at 133.35 165.1 0) (unit 1)
 		(property "Reference" "Q2" (at 123.19 161.29 0) (effects (font (size 1.27 1.27))))
 		(property "Value" "AO3401A" (at 123.19 168.91 0) (effects (font (size 1.27 1.27))))
