File: hw/.history/teacup-carrier-merge-test.kicad_pcb (KiCad board)
At the start: 4 copper layers, 257 x 117.5 mm, 137 parts, among them J1 AH58893-T9B10-3F, J2 TYPE-C-31-M-12, J20 HDR_J20, J21 HDR_J21, J22 HDR_J22, J23 HDR_J23, J24 HDR_J24, J25 HDR_J25, J26 HDR_J26, J27 HDR_J27, J28 HDR_J28, J29 HDR_J29, J3 TE_292303-7, J30 HDR_J30, J31 HDR_J31, J32 HDR_J32, J33 HDR_J33, J34 HDR_J34, J35 HDR_J35, J36 HDR_J36, J37 HDR_J37, J38 AMP_MIC_TAP, J4 Hirose_DM3D-SF, J5 Wuerth_694106301002, J6 AudioJack4_Ground, J7 SFW15R-2STE1LF, J8 SFW15R-2STE1LF, J9 TYPE-C-31-M-12, Q1 AO3401A, Q2 AO3401A, SW1 SSSS711403, SW2 SSSS711403, U1 AP62600SJ-7, U10 TS5A3166, U11 DIP-8 Socket, U12 TPS2053BDR, U13 W25Q32JVSS, U14 TPS22990DMLR, U15 TCA9555PWR, U2 AP62300WU-7, U3 MCP4661-104E_ST, U4 TPS22990DMLR, U5 AZ1117CH-3.3TRG1, U6 AZ1117CH-1.8TRG1, U7 AP62300WU-7, U8 ESP32-S3-WROOM-1-N16R2, U9 TS5A3166

Commit message: Add MSC1 breakout (J37), ground J35 spare pads, add audio amp/mic tap (J38)
Carve J35's last 6 pins into a new MSC1 header (J37: CLK/CMD/D0-D3_CD),
keeping J35 at a fixed 26-pin size in both schematic and PCB with the
now-orphaned pads tied to GND. Add a 3-pin tap (J38) off the audio jack
(HPOUTL/GND/MICLP) so an external amplifier or mic can be wired in
directly instead of needing a breakout cable off J6.
Parts:
- removed J37: HDR_J37, PinHeader_1x07_P2.54mm_Vertical
- removed J38: AMP_MIC_TAP, PinHeader_1x03_P2.54mm_Vertical
Connections:
- J1 pad 283: MSC1_CLK -> SPARE_P283
- J1 pad 284: MSC1_CMD -> SPARE_P284
- J1 pad 285: MSC1_D0 -> SPARE_P285
- J1 pad 286: MSC1_D1 -> SPARE_P286
- J1 pad 287: MSC1_D2 -> SPARE_P287
- J1 pad 288: MSC1_D3_CD -> SPARE_P288
- J35 pad 20: GND -> SPARE_P283
- J35 pad 21: GND -> SPARE_P284
- J35 pad 22: GND -> SPARE_P285
- J35 pad 23: GND -> SPARE_P286
- J35 pad 24: GND -> SPARE_P287
- J35 pad 25: GND -> SPARE_P288
Other:
- board text removed: "AMP/MIC"
- board text removed: "MSC1"
- board text removed: "UART1"
