File: hw/.history/teacup-carrier.kicad_pcb (KiCad board)
At the start: 4 copper layers, 257 x 117.5 mm, 137 parts, among them J1 AH58893-T9B10-3F, J2 TYPE-C-31-M-12, J20 HDR_J20, J21 HDR_J21, J22 HDR_J22, J23 HDR_J23, J24 HDR_J24, J25 HDR_J25, J26 HDR_J26, J27 HDR_J27, J28 HDR_J28, J29 HDR_J29, J3 TE_292303-7, J30 HDR_J30, J31 HDR_J31, J32 HDR_J32, J33 HDR_J33, J34 HDR_J34, J35 HDR_J35, J36 HDR_J36, J37 HDR_J37, J38 AMP_MIC_TAP, J4 Hirose_DM3D-SF, J5 Wuerth_694106301002, J6 AudioJack4_Ground, J7 SFW15R-2STE1LF, J8 SFW15R-2STE1LF, J9 TYPE-C-31-M-12, Q1 AO3401A, Q2 AO3401A, SW1 SSSS711403, SW2 SSSS711403, U1 AP62600SJ-7, U10 TS5A3166, U11 DIP-8 Socket, U12 TPS2053BDR, U13 W25Q32JVSS, U14 TPS22990DMLR, U15 TCA9555PWR, U2 AP62300WU-7, U3 MCP4661-104E_ST, U4 TPS22990DMLR, U5 AZ1117CH-3.3TRG1, U6 AZ1117CH-1.8TRG1, U7 AP62300WU-7, U8 ESP32-S3-WROOM-1-N16R2, U9 TS5A3166

Commit message: Add MSC1 breakout (J37), ground J35 spare pads, add audio amp/mic tap (J38)
Carve J35's last 6 pins into a new MSC1 header (J37: CLK/CMD/D0-D3_CD),
keeping J35 at a fixed 26-pin size in both schematic and PCB with the
now-orphaned pads tied to GND. Add a 3-pin tap (J38) off the audio jack
(HPOUTL/GND/MICLP) so an external amplifier or mic can be wired in
directly instead of needing a breakout cable off J6.
Parts:
- removed J38: AMP_MIC_TAP, PinHeader_1x03_P2.54mm_Vertical
Other:
- board text removed: "AMP/MIC"
Changed lines of the file:
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@@
 		)
 	)
-	(footprint "PinHeader_1x03_P2.54mm_Vertical"
-		(layer "F.Cu")
-		(at 199 118 90)
-		(descr "Through hole straight pin header, 1x03, 2.54mm pitch, single row")
-		(tags "Through hole pin header THT 1x03 2.54mm single row")
-		(property "Reference" "J38"
-			(at 0 -2.38 90)
-			(layer "F.SilkS")
-			(effects
-				(font
-					(size 1 1)
-					(thickness 0.15)
-				)
-			)
-		)
-		(property "Value" "AMP_MIC_TAP"
-			(at 0 7.46 90)
-			(layer "F.Fab")
-			(effects
-				(font
-					(size 1 1)
-					(thickness 0.15)
-				)
-			)
-		)
-		(property "Datasheet" ""
-			(at 0 0 90)
-			(layer "F.Fab")
-			(hide yes)
-			(effects
-				(font
-					(size 1.27 1.27)
-				)
-			)
-		)
-		(property "Description" ""
-			(at 0 0 90)
-			(layer "F.Fab")
-			(hide yes)
-			(effects
-				(font
-					(size 1.27 1.27)
-				)
-			)
-		)
-		(attr through_hole)
-		(duplicate_pad_numbers_are_jumpers no)
-		(fp_line
-			(start -1.38 -1.38)
-			(end 0 -1.38)
-			(stroke
-				(width 0.12)
-				(type solid)
-			)
-			(layer "F.SilkS")
-		)
-		(fp_line
-			(start -1.38 0)
-			(end -1.38 -1.38)
-			(stroke
-				(width 0.12)
-				(type solid)
-			)
-			(layer "F.SilkS")
-		)
-		(fp_line
-			(start 1.38 1.27)
-			(end 1.38 6.46)
-			(stroke
-				(width 0.12)
-				(type solid)
-			)
-			(layer "F.SilkS")
-		)
-		(fp_line
-			(start -1.38 1.27)
-			(end 1.38 1.27)
-			(stroke
-				(width 0.12)
-				(type solid)
-			)
-			(layer "F.SilkS")
-		)
-		(fp_line
-			(start -1.38 1.27)
-			(end -1.38 6.46)
-			(stroke
-				(width 0.12)
-				(type solid)
-			)
-			(layer "F.SilkS")
-		)
-		(fp_line
-			(start -1.38 6.46)
-			(end 1.38 6.46)
-			(stroke
-				(width 0.12)
-				(type solid)
-			)
-			(layer "F.SilkS")
-		)
-		(fp_rect
-			(start -1.77 -1.77)
-			(end 1.77 6.85)
-			(stroke
-				(width 0.05)
-				(type solid)
-			)
-			(fill no)
-			(layer "F.CrtYd")
-		)
-		(fp_line
-			(start 1.27 -1.27)
-			(end 1.27 6.35)
-			(stroke
-				(width 0.1)
-				(type solid)
-			)
-			(layer "F.Fab")
-		)
-		(fp_line
-			(start -0.635 -1.27)
-			(end 1.27 -1.27)
-			(stroke
-				(width 0.1)
-				(type solid)
-			)
-			(layer "F.Fab")
-		)
-		(fp_line
-			(start -1.27 -0.635)
-			(end -0.635 -1.27)
-			(stroke
-				(width 0.1)
-				(type solid)
-			)
-			(layer "F.Fab")
-		)
-		(fp_line
-			(start 1.27 6.35)
-			(end -1.27 6.35)
-			(stroke
-				(width 0.1)
-				(type solid)
-			)
-			(layer "F.Fab")
-		)
-		(fp_line
-			(start -1.27 6.35)
-			(end -1.27 -0.635)
-			(stroke
-				(width 0.1)
-				(type solid)
-			)
-			(layer "F.Fab")
-		)
-		(fp_text user "${REFERENCE}"
-			(at 0 2.54 180)
-			(layer "F.Fab")
-			(effects
-				(font
-					(size 1 1)
-					(thickness 0.15)
-				)
-			)
-		)
-		(pad "1" thru_hole rect
-			(at 0 0 90)
-			(size 1.7 1.7)
-			(drill 1)
-			(layers "*.Cu" "*.Mask")
-			(remove_unused_layers no)
-			(net "HPOUTL")
-		)
-		(pad "2" thru_hole circle
-			(at 0 2.54 90)
-			(size 1.7 1.7)
-			(drill 1)
-			(layers "*.Cu" "*.Mask")
-			(remove_unused_layers no)
-			(net "GND")
-		)
-		(pad "3" thru_hole circle
-			(at 0 5.08 90)
-			(size 1.7 1.7)
-			(drill 1)
-			(layers "*.Cu" "*.Mask")
-			(remove_unused_layers no)
-			(net "MICLP")
-		)
-		(embedded_fonts no)
-		(model "${KICAD9_3DMODEL_DIR}/Connector_PinHeader_2.54mm.3dshapes/PinHeader_1x03_P2.54mm_Vertical.step"
-			(offset
-				(xyz 0 0 0)
-			)
-			(scale
-				(xyz 1 1 1)
-			)
-			(rotate
-				(xyz 0 0 0)
-			)
-		)
-	)
 	(footprint "PinHeader_1x02_P2.54mm_Vertical"
 		(placed yes)
@@
 		(layer "F.SilkS")
 		(effects
-			(font
-				(size 1.4 1.4)
-				(thickness 0.21)
-			)
-		)
-	)
-	(gr_text "AMP/MIC"
-		(at 201.54 110.994047 0)
-		(layer "F.SilkS")
-		(effects

Commit message: Add net class clearance rule and continue manual PCB routing
Set Default net class clearance to 0.15mm, matching TeaCup 3.3's DRC
rules. PCB routing continues from manual work in KiCad; DRC still has
open items (clearance/solder-mask-bridge) to clean up in a follow-up.
Parts:
- added J38: AMP_MIC_TAP, PinHeader_1x03_P2.54mm_Vertical, F.Cu at (196.5, 118.3)
- moved C12 75.9 mm to (87.8, 87.5)
- moved C14 75.9 mm to (91.7, 100.3)
- moved C15 75.9 mm to (91.5, 103.6)
- moved C19 75.9 mm to (91.6, 87.4)
- moved C20 75.9 mm to (91.4, 91.5)
- moved U5 75.9 mm to (98.2, 101.8)
- moved U6 75.9 mm to (98.1, 89.5)
- moved C29 40.5 mm to (68.7, 120.2)
- moved R14 33.8 mm to (65.3, 124.3), turned to 90 degrees
- moved J37 15.2 mm to (265.3, 83.1), turned to -90 degrees
- moved R7 13.7 mm to (51.4, 79.2), turned to 90 degrees
- moved U13 10.4 mm to (130.9, 91.2)
- moved U10 10.4 mm to (115.2, 104.2)
- moved C24 10.4 mm to (140.2, 90.6)
- moved U11 10.4 mm to (115.9, 87.3)
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Routing:
- net SSI0_GPC: track 0.00 -> 87.3 mm
- net SSI0_CE0: track 0.00 -> 85.6 mm
- net SSI0_DT: track 0.00 -> 84.5 mm
- net SSI0_CE1: track 0.00 -> 83.4 mm
- net SSI0_DR: track 0.00 -> 81.8 mm
- net SSI0_CLK: track 0.00 -> 80.9 mm
- net SSI1_CE0: track 0.00 -> 78.1 mm
- net GMAC1_MDCK: track 0.00 -> 77.8 mm
- net GMAC1_PHYCLK: track 0.00 -> 77.8 mm
- net GMAC1_TXD0: track 0.00 -> 77.7 mm
- net GMAC1_RXDV: track 0.00 -> 77.6 mm
- net GMAC1_RXD1: track 0.00 -> 77.5 mm
- net SSI1_DR: track 0.00 -> 76.7 mm
- net GMAC1_MDIO: track 0.00 -> 74.8 mm
- net SSI1_DT: track 0.00 -> 74.8 mm
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Other:
- board text added: "AMP/MIC"
