File: hw/.history/teacup-carrier.kicad_pcb (KiCad board)
At the start: 4 copper layers, 257 x 117.5 mm, 137 parts, among them J1 AH58893-T9B10-3F, J2 TYPE-C-31-M-12, J20 HDR_J20, J21 HDR_J21, J22 HDR_J22, J23 HDR_J23, J24 HDR_J24, J25 HDR_J25, J26 HDR_J26, J27 HDR_J27, J28 HDR_J28, J29 HDR_J29, J3 TE_292303-7, J30 HDR_J30, J31 HDR_J31, J32 HDR_J32, J33 HDR_J33, J34 HDR_J34, J35 HDR_J35, J36 HDR_J36, J37 HDR_J37, J38 AMP_MIC_TAP, J4 Hirose_DM3D-SF, J5 Wuerth_694106301002, J6 AudioJack4_Ground, J7 SFW15R-2STE1LF, J8 SFW15R-2STE1LF, J9 TYPE-C-31-M-12, Q1 AO3401A, Q2 AO3401A, SW1 SSSS711403, SW2 SSSS711403, U1 AP62600SJ-7, U10 TS5A3166, U11 DIP-8 Socket, U12 TPS2053BDR, U13 W25Q32JVSS, U14 TPS22990DMLR, U15 TCA9555PWR, U2 AP62300WU-7, U3 MCP4661-104E_ST, U4 TPS22990DMLR, U5 AZ1117CH-3.3TRG1, U6 AZ1117CH-1.8TRG1, U7 AP62300WU-7, U8 ESP32-S3-WROOM-1-N16R2, U9 TS5A3166

Commit message: Fix schematic<->PCB linking, reorder J1 pins by connected peer, add +3V3 plane, wire microSD card-detect
- schgen.py: deterministic per-symbol UUIDs (uuid5, keyed on ref designator)
  instead of random uuid4, so PCB footprints stay linked to their schematic
  symbol across regenerations; link all 133 real PCB footprints to their
  schematic symbol via path, fixing "Update PCB from Schematic" placing
  duplicates.
- J1 pin reorg: audio (HPOUTL/MICLP) moved from 170/171 to 6/7 (170/171 now
  GND); USBA_HOST_DP/DM moved from 40/41 to 20/21 (40/41 now GND); the 20
  pins connected directly to U8 (ESP32-S3) reordered so U8's ascending pin
  number maps to J1's descending pin number; +5V_MODEA (redundant -- a
  self-contained module already needs its own bare-bench power input)
  replaced with +5V_SW (the real arbitrated switched-5V rail) on pins 17/18.
- New +3V3 copper pour on In1.Cu, mirroring the existing GND pour; every
  +3V3 pad on the board (38, now 39 with R43) gets a stub trace + via down
  to it.
- microSD (J4): switched to the Micro_SD_Card_Det2 symbol so pin 10 (the
  footprint's real card-detect pad) has somewhere to attach; added R43
  (1M, matches TeaCup 3.3's R22) pulling MSC0_CD up to +3V3.
- fp-lib-table: replaced hardcoded /usr/share/kicad/footprints/... paths
  with ${KICAD10_FOOTPRINT_DIR}, fixing "footprint not found" errors for
  every component when Update PCB from Schematic runs outside this Linux
  environment.

Verified throughout via isolated ERC/DRC diffs against pre-change
baselines; each change confirmed to produce only its own intended delta.
Parts:
- added R43: 1M, Resistor_SMD:R_0402_1005Metric, F.Cu at (196.3, 126.5)
- C1, C10, C11, C15, C16, C18, C20, C21, C27, C28, C29, C6, C9: footprint C_0805_2012Metric -> Capacitor_SMD:C_0805_2012Metric
- C12, C13, C17, C2, C22, C23, C24, C25, C26, C3, C4, C5, C7: footprint C_0402_1005Metric -> Capacitor_SMD:C_0402_1005Metric
- C14, C19: footprint C_0603_1608Metric -> Capacitor_SMD:C_0603_1608Metric
- D1, D2: footprint Nexperia_CFP3_SOD-123W -> Diode_SMD:Nexperia_CFP3_SOD-123W
- J1: footprint DDR4288S0511H_UDIMM288 -> teacup-carrier:DDR4288S0511H_UDIMM288
- J2, J9: footprint USB_C_Receptacle_HRO_TYPE-C-31-M-12 -> Connector_USB:USB_C_Receptacle_HRO_TYPE-C-31-M-12
- J20, J21: footprint PinHeader_2x06_P2.54mm_Vertical -> Connector_PinHeader_2.54mm:PinHeader_2x06_P2.54mm_Vertical
- J22, J23, J24, J26, J29: footprint PinHeader_1x05_P2.54mm_Vertical -> Connector_PinHeader_2.54mm:PinHeader_1x05_P2.54mm_Vertical
- J25: footprint PinHeader_2x04_P2.54mm_Vertical -> Connector_PinHeader_2.54mm:PinHeader_2x04_P2.54mm_Vertical
- J27: footprint PinHeader_2x05_P2.54mm_Vertical -> Connector_PinHeader_2.54mm:PinHeader_2x05_P2.54mm_Vertical
- J28, JP10, JP2, JP3, JP4, JP5, JP6, JP7, JP8, JP9: footprint PinHeader_1x02_P2.54mm_Vertical -> Connector_PinHeader_2.54mm:PinHeader_1x02_P2.54mm_Vertical
- J3: footprint USB_A_TE_292303-7_Horizontal -> Connector_USB:USB_A_TE_292303-7_Horizontal
- J30: footprint PinHeader_2x09_P2.54mm_Vertical -> Connector_PinHeader_2.54mm:PinHeader_2x09_P2.54mm_Vertical
- J31: footprint PinHeader_2x11_P2.54mm_Vertical -> Connector_PinHeader_2.54mm:PinHeader_2x11_P2.54mm_Vertical
- J32, J33, J34, J35: footprint PinHeader_2x13_P2.54mm_Vertical -> Connector_PinHeader_2.54mm:PinHeader_2x13_P2.54mm_Vertical
- J36, J38: footprint PinHeader_1x03_P2.54mm_Vertical -> Connector_PinHeader_2.54mm:PinHeader_1x03_P2.54mm_Vertical
- J37: footprint PinHeader_1x07_P2.54mm_Vertical -> Connector_PinHeader_2.54mm:PinHeader_1x07_P2.54mm_Vertical
- J4: footprint microSD_HC_Hirose_DM3D-SF -> Connector_Card:microSD_HC_Hirose_DM3D-SF
- J5: footprint BarrelJack_Wuerth_6941xx301002 -> Connector_BarrelJack:BarrelJack_Wuerth_6941xx301002
- J6: footprint Jack_3.5mm_PJ320D_Horizontal -> Connector_Audio:Jack_3.5mm_PJ320D_Horizontal
- J7, J8: footprint FPC-SMD_15P-P1.00_SFW15R-2STE1LF -> teacup-carrier:FPC-SMD_15P-P1.00_SFW15R-2STE1LF
- JP11, JP12: footprint PinHeader_1x03_P2.54mm_Vertical_SMD_Pin1Left -> Connector_PinHeader_2.54mm:PinHeader_1x03_P2.54mm_Vertical_SMD_Pin1Left
- L1, L2, L3: footprint L_1210_3225Metric -> Inductor_SMD:L_1210_3225Metric
- Q1, Q2: footprint SOT-23 -> Package_TO_SOT_SMD:SOT-23
- R1, R10, R11, R12, R13, R14, R15, R16, R17, R18, R19, R2, R20, R21, R22, R23, R24, R25, R26, R27, R28, R29, R3, R30, R31, R32, R33, R34, R35, R36, R37, R38, R39, R4, R40, R41, R42, R5, R6, R7, R8, R9: footprint R_0402_1005Metric -> Resistor_SMD:R_0402_1005Metric
- SW1, SW2: footprint SW-TH_SSSS711403 -> teacup-carrier:SW-TH_SSSS711403
- U1: footprint QFN-12_L3.0-W2.0-P0.50-TL_AP62600SJ-7 -> teacup-carrier:QFN-12_L3.0-W2.0-P0.50-TL_AP62600SJ-7
- U10, U9: footprint SOT-23-5 -> Package_TO_SOT_SMD:SOT-23-5
- U11: footprint DIP-8_W7.62mm_Socket -> Package_DIP:DIP-8_W7.62mm_Socket
- U12: footprint SOIC-16_3.9x9.9mm_P1.27mm -> Package_SO:SOIC-16_3.9x9.9mm_P1.27mm
- U13: footprint SOIC-8_5.3x5.3mm_P1.27mm -> Package_SO:SOIC-8_5.3x5.3mm_P1.27mm
- U14, U4: footprint WSON-10_L3.0-W2.0-P0.50-BL-EP_TI_DML -> teacup-carrier:WSON-10_L3.0-W2.0-P0.50-BL-EP_TI_DML
- U15: footprint TSSOP-24_4.4x7.8mm_P0.65mm -> Package_SO:TSSOP-24_4.4x7.8mm_P0.65mm
- U2, U7: footprint TSOT-23-6_L2.9-W1.6-P0.95-LS2.8-BL -> teacup-carrier:TSOT-23-6_L2.9-W1.6-P0.95-LS2.8-BL
- U3: footprint TSSOP-14_4.4x5mm_P0.65mm -> Package_SO:TSSOP-14_4.4x5mm_P0.65mm
- U5, U6: footprint SOT-223-3_TabPin2 -> Package_TO_SOT_SMD:SOT-223-3_TabPin2
- U8: footprint ESP32-S3-WROOM-1 -> teacup-carrier:ESP32-S3-WROOM-1
- moved J6 215.3 mm to (25.9, 48.1), turned to 0 degrees
- moved J38 193.9 mm to (41.2, 45.5), turned to 0 degrees
- moved C22 105.6 mm to (46.2, 138.8)
- moved R10 105.6 mm to (55.8, 135.2)
- moved R8 105.6 mm to (45.4, 130.0)
- moved C13 105.6 mm to (63.0, 131.5)
- moved C16 105.6 mm to (51.8, 127.4)
- moved C2 105.6 mm to (59.5, 131.4)
- moved R11 105.6 mm to (67.8, 133.5)
- moved R21 105.6 mm to (58.9, 124.6)
- moved R4 105.6 mm to (56.5, 127.9)
- moved C1 105.6 mm to (56.3, 131.4)
- moved C21 105.6 mm to (46.2, 134.4)
- moved C6 105.6 mm to (51.7, 131.4)
- moved D1 105.6 mm to (62.6, 123.8)
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Connections:
- J1 pad 17: +5V_MODEA -> +5V_SW
- J1 pad 170: HPOUTL -> GND
- J1 pad 171: MICLP -> GND
- J1 pad 18: +5V_MODEA -> +5V_SW
- J1 pad 20: GND -> USBA_HOST_DP
- J1 pad 21: GND -> USBA_HOST_DM
- J1 pad 23: I2C_ID_SDA -> VCORE_SNS
- J1 pad 24: I2C_ID_SCL -> HOSTED_DATA_READY
- J1 pad 25: VCORE_SNS -> HOSTED_HANDSHAKE
- J1 pad 26: BOOTSEL -> HOSTED_SPI_CS
- J1 pad 27: RESET_EN -> HOSTED_SPI_MISO
- J1 pad 28: SFC_CS -> SFC_IO2
- J1 pad 29: SFC_CLK -> SFC_IO1
- J1 pad 30: SFC_IO0 -> SFC_CLK
- J1 pad 31: SFC_IO1 -> SFC_IO0
- J1 pad 32: SFC_IO2 -> SFC_CS
- J1 pad 34: UART1_TX -> RESET_EN
- J1 pad 35: UART1_RX -> BOOTSEL
- J1 pad 40: USBA_HOST_DP -> GND
- J1 pad 41: USBA_HOST_DM -> GND
- J1 pad 42: HOSTED_RESET -> UART1_RX
- J1 pad 43: HOSTED_SPI_CLK -> UART1_TX
- J1 pad 45: HOSTED_SPI_MISO -> HOSTED_SPI_CLK
- J1 pad 46: HOSTED_SPI_CS -> I2C_ID_SCL
- J1 pad 47: HOSTED_HANDSHAKE -> I2C_ID_SDA
- J1 pad 48: HOSTED_DATA_READY -> HOSTED_RESET
- J1 pad 6: GND -> MICLP
- J1 pad 60: MIPI0_GPIO -> MIPI0_SCCB_SDA
- J1 pad 61: MIPI0_SCCB_SDA -> MIPI0_SCCB_SCL
- J1 pad 62: MIPI0_SCCB_SCL -> MIPI0_GPIO
- J1 pad 7: GND -> HPOUTL
- J4 pad 10: (no net) -> MSC0_CD
Routing:
- net MSC0_D1: track 0.00 -> 131.2 mm
- net MSC0_D0: track 0.00 -> 130.0 mm
- net MSC0_CLK: track 0.00 -> 128.2 mm
- net MSC0_CMD: track 0.00 -> 126.2 mm
- net MIPI0_SCCB_SCL: track 0.00 -> 125.6 mm
- net MIPI0_SCCB_SDA: track 0.00 -> 125.6 mm
- net MSC0_D3_CD: track 0.00 -> 125.2 mm
- net MSC0_D2: track 0.00 -> 124.6 mm
- net MIPI0_CLKP: track 39.5 -> 125.5 mm
- net MIPI0_CLKN: track 39.5 -> 125.5 mm
- net MIPI0_D1P: track 39.7 -> 125.6 mm
- net MIPI0_D1N: track 39.7 -> 125.5 mm
- net MIPI0_D0P: track 39.8 -> 125.6 mm
- net MIPI0_D0N: track 39.9 -> 125.6 mm
- net MIPI1_CLKN: track 41.8 -> 125.5 mm
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- added copper zone on In1.Cu, net +3V3
