File: hw/.history/teacup-carrier.kicad_sch (KiCad schematic)
At the start: 80 parts, among them J1 AH58893-T9B10-3F, J2 TYPE-C-31-M-12, J3 TE_292303-7, J4 Hirose_DM3D-SF, J5 Wuerth_694106301002, J6 AudioJack4_Ground, J7 SFW15R-2STE1LF, J8 SFW15R-2STE1LF, J9 TYPE-C-31-M-12, Q1 AO3401A, Q2 AO3401A, SW1 SSSS711403, SW2 SSSS711403, U1 AP62600SJ-7, U10 TS5A3166, U11 DIP-8 Socket, U12 TPS2053BDR, U13 W25Q32JVSS, U14 TPS22990DMLR, U15 TCA9555PWR, U2 AP62300WU-7, U3 MCP4661-104E_ST, U4 TPS22990DMLR, U5 AZ1117CH-3.3TRG1, U6 AZ1117CH-1.8TRG1, U7 AP62300WU-7, U8 ESP32-S3-WROOM-1-N16R2, U9 TS5A3166

Commit message: Add MSC1 breakout (J37), ground J35 spare pads, add audio amp/mic tap (J38)
Carve J35's last 6 pins into a new MSC1 header (J37: CLK/CMD/D0-D3_CD),
keeping J35 at a fixed 26-pin size in both schematic and PCB with the
now-orphaned pads tied to GND. Add a 3-pin tap (J38) off the audio jack
(HPOUTL/GND/MICLP) so an external amplifier or mic can be wired in
directly instead of needing a breakout cable off J6.
Parts:
- removed JP1: PROVISIONED, Connector_PinHeader_2.54mm:PinHeader_1x02_P2.54mm_Vertical, symbol Connector_Generic:Conn_01x02
- added C24, C25, C26: 100nF, Capacitor_SMD:C_0402_1005Metric, symbol Device:C
- added C27, C28, C29: 10uF, Capacitor_SMD:C_0805_2012Metric, symbol Device:C
- added J20: HDR_J20, Connector_PinHeader_2.54mm:PinHeader_1x11_P2.54mm_Vertical, symbol Connector_Generic:Conn_01x11
- added J21: HDR_J21, Connector_PinHeader_2.54mm:PinHeader_1x11_P2.54mm_Vertical, symbol Connector_Generic:Conn_01x11
- added J22: HDR_J22, Connector_PinHeader_2.54mm:PinHeader_1x05_P2.54mm_Vertical, symbol Connector_Generic:Conn_01x05
- added J23: HDR_J23, Connector_PinHeader_2.54mm:PinHeader_1x05_P2.54mm_Vertical, symbol Connector_Generic:Conn_01x05
- added J24: HDR_J24, Connector_PinHeader_2.54mm:PinHeader_1x05_P2.54mm_Vertical, symbol Connector_Generic:Conn_01x05
- added J25: HDR_J25, Connector_PinHeader_2.54mm:PinHeader_1x07_P2.54mm_Vertical, symbol Connector_Generic:Conn_01x07
- added J26: HDR_J26, Connector_PinHeader_2.54mm:PinHeader_1x05_P2.54mm_Vertical, symbol Connector_Generic:Conn_01x05
- added J27: HDR_J27, Connector_PinHeader_2.54mm:PinHeader_1x09_P2.54mm_Vertical, symbol Connector_Generic:Conn_01x09
- added J28: HDR_J28, Connector_PinHeader_2.54mm:PinHeader_1x02_P2.54mm_Vertical, symbol Connector_Generic:Conn_01x02
- added J29: HDR_J29, Connector_PinHeader_2.54mm:PinHeader_1x05_P2.54mm_Vertical, symbol Connector_Generic:Conn_01x05
- added J30: HDR_J30, Connector_PinHeader_2.54mm:PinHeader_1x17_P2.54mm_Vertical, symbol Connector_Generic:Conn_01x17
- added J31: HDR_J31, Connector_PinHeader_2.54mm:PinHeader_1x24_P2.54mm_Vertical, symbol Connector_Generic:Conn_01x24
- added J32: HDR_J32, Connector_PinHeader_2.54mm:PinHeader_1x25_P2.54mm_Vertical, symbol Connector_Generic:Conn_01x25
- added J33: HDR_J33, Connector_PinHeader_2.54mm:PinHeader_1x25_P2.54mm_Vertical, symbol Connector_Generic:Conn_01x25
- added J34: HDR_J34, Connector_PinHeader_2.54mm:PinHeader_1x25_P2.54mm_Vertical, symbol Connector_Generic:Conn_01x25
- added J35: HDR_J35, Connector_PinHeader_2.54mm:PinHeader_1x25_P2.54mm_Vertical, symbol Connector_Generic:Conn_01x25
- added JP10, JP6: COMPUTER, Connector_PinHeader_2.54mm:PinHeader_1x02_P2.54mm_Vertical, symbol Connector_Generic:Conn_01x02
- added JP2: 0.8V, Connector_PinHeader_2.54mm:PinHeader_1x02_P2.54mm_Vertical, symbol Connector_Generic:Conn_01x02
- added JP3: 0.9V, Connector_PinHeader_2.54mm:PinHeader_1x02_P2.54mm_Vertical, symbol Connector_Generic:Conn_01x02
- added JP4: 1.0V, Connector_PinHeader_2.54mm:PinHeader_1x02_P2.54mm_Vertical, symbol Connector_Generic:Conn_01x02
- added JP5: 1.1V, Connector_PinHeader_2.54mm:PinHeader_1x02_P2.54mm_Vertical, symbol Connector_Generic:Conn_01x02
- added JP7: 1.35V, Connector_PinHeader_2.54mm:PinHeader_1x02_P2.54mm_Vertical, symbol Connector_Generic:Conn_01x02
- added JP8: 1.5V, Connector_PinHeader_2.54mm:PinHeader_1x02_P2.54mm_Vertical, symbol Connector_Generic:Conn_01x02
- added JP9: 1.8V, Connector_PinHeader_2.54mm:PinHeader_1x02_P2.54mm_Vertical, symbol Connector_Generic:Conn_01x02
- added R25, R26, R41, R42: 4.7k, Resistor_SMD:R_0402_1005Metric, symbol Device:R
- added R27: 3.32k, Resistor_SMD:R_0402_1005Metric, symbol Device:R
- added R28, R30, R32, R34, R36, R38, R40: 10.0k, Resistor_SMD:R_0402_1005Metric, symbol Device:R
- added R29: 4.99k, Resistor_SMD:R_0402_1005Metric, symbol Device:R
- added R31: 6.65k, Resistor_SMD:R_0402_1005Metric, symbol Device:R
- added R33: 8.25k, Resistor_SMD:R_0402_1005Metric, symbol Device:R
- added R35: 6.81k, Resistor_SMD:R_0402_1005Metric, symbol Device:R
- added R37: 8.66k, Resistor_SMD:R_0402_1005Metric, symbol Device:R
- added R39: 12.4k, Resistor_SMD:R_0402_1005Metric, symbol Device:R
Connections:
- net SW2_POLE is gone; now on net +5V_ALT: SW2.3
- net USB1_VBUS_IN is gone; now on net +5V_SW: U12.2 (IN1)
- net USB2_VBUS_IN is gone; now on net +5V_SW: U12.6 (IN2)
- net +3V3: now also C24.1, C25.1, C26.1, R25.1, R26.1, R41.1, R42.1; no longer R5.1
- net +5V_ALT: now also C28.1
- net +5V_BMC: now also C27.1
- net +5V_SW: now also R5.1
- net DCJACK_VBUS: now also C29.1
- net GND: now also J1.102 (P102), J1.107 (P107), J1.112 (P112), J1.123 (P123), J1.130 (P130), J1.135 (P135), J1.144 (P144), J1.145 (P145), J1.147 (P147), J1.152 (P152), J1.169 (P169), J1.97 (P97), C24.2, C25.2, C26.2, C27.2, C28.2, C29.2, J20.1 (Pin_1), J21.1 (Pin_1), J22.1 (Pin_1), J23.1 (Pin_1), J24.1 (Pin_1), J25.1 (Pin_1), J26.1 (Pin_1), J27.1 (Pin_1), J28.1 (Pin_1), J29.1 (Pin_1), J30.1 (Pin_1), J31.1 (Pin_1), J32.1 (Pin_1), J33.1 (Pin_1), J34.1 (Pin_1), J35.1 (Pin_1), R28.2, R30.2, R32.2, R34.2, R36.2, R38.2, R40.2
- net I2C_ID_SCL: now also R42.2
- net I2C_ID_SDA: now also R41.2
- net I2C_PWR_SCL: now also R26.2
- net I2C_PWR_SDA: now also R25.2
- net VCORE: now also R27.1, R29.1, R31.1, R33.1
- net VDDR: now also R35.1, R37.1, R39.1
- net SPARE_P193: now reaches J1.193 (P193)
- net SPARE_P193: now also J32.2 (Pin_2)
- net SPARE_P194: now reaches J1.194 (P194)
- net SPARE_P194: now also J32.3 (Pin_3)
- net SPARE_P195: now reaches J1.195 (P195)
- net SPARE_P195: now also J32.4 (Pin_4)
- net SPARE_P196: now reaches J1.196 (P196)
- net SPARE_P196: now also J32.5 (Pin_5)
- net SPARE_P197: now reaches J1.197 (P197)
- net SPARE_P197: now also J32.6 (Pin_6)
- net SPARE_P198: now reaches J1.198 (P198)
- net SPARE_P198: now also J32.7 (Pin_7)
- net SPARE_P199: now reaches J1.199 (P199)
- net SPARE_P199: now also J32.8 (Pin_8)
- net SPARE_P200: now reaches J1.200 (P200)
- net SPARE_P200: now also J32.9 (Pin_9)
- net SPARE_P201: now reaches J1.201 (P201)
- net SPARE_P201: now also J32.10 (Pin_10)
- net SPARE_P202: now reaches J1.202 (P202)
- net SPARE_P202: now also J32.11 (Pin_11)
- net SPARE_P203: now reaches J1.203 (P203)
- net SPARE_P203: now also J32.12 (Pin_12)
- net SPARE_P204: now reaches J1.204 (P204)
- net SPARE_P204: now also J32.13 (Pin_13)
- net SPARE_P205: now reaches J1.205 (P205)
- net SPARE_P205: now also J32.14 (Pin_14)
- net SPARE_P206: now reaches J1.206 (P206)
- net SPARE_P206: now also J32.15 (Pin_15)
- net SPARE_P207: now reaches J1.207 (P207)
- net SPARE_P207: now also J32.16 (Pin_16)
- net SPARE_P208: now reaches J1.208 (P208)
- net SPARE_P208: now also J32.17 (Pin_17)
- net SPARE_P209: now reaches J1.209 (P209)
- net SPARE_P209: now also J32.18 (Pin_18)
- net SPARE_P210: now reaches J1.210 (P210)
- net SPARE_P210: now also J32.19 (Pin_19)
- net SPARE_P211: now reaches J1.211 (P211)
- net SPARE_P211: now also J32.20 (Pin_20)
- net SPARE_P212: now reaches J1.212 (P212)
- net SPARE_P212: now also J32.21 (Pin_21)
- net SPARE_P213: now reaches J1.213 (P213)
- net SPARE_P213: now also J32.22 (Pin_22)
- net SPARE_P214: now reaches J1.214 (P214)
- net SPARE_P214: now also J32.23 (Pin_23)
- net SPARE_P215: now reaches J1.215 (P215)
- net SPARE_P215: now also J32.24 (Pin_24)
- net SPARE_P216: now reaches J1.216 (P216)
- net SPARE_P216: now also J32.25 (Pin_25)
- net SPARE_P217: now reaches J1.217 (P217)
- net SPARE_P217: now also J33.2 (Pin_2)
- net SPARE_P218: now reaches J1.218 (P218)
- net SPARE_P218: now also J33.3 (Pin_3)
- net SPARE_P219: now reaches J1.219 (P219)
- net SPARE_P219: now also J33.4 (Pin_4)
- net SPARE_P220: now reaches J1.220 (P220)
- net SPARE_P220: now also J33.5 (Pin_5)
- net SPARE_P221: now reaches J1.221 (P221)
- net SPARE_P221: now also J33.6 (Pin_6)
- net SPARE_P222: now reaches J1.222 (P222)
- net SPARE_P222: now also J33.7 (Pin_7)
- net SPARE_P223: now reaches J1.223 (P223)
- net SPARE_P223: now also J33.8 (Pin_8)
- net SPARE_P224: now reaches J1.224 (P224)
- net SPARE_P224: now also J33.9 (Pin_9)
- net SPARE_P225: now reaches J1.225 (P225)
- net SPARE_P225: now also J33.10 (Pin_10)
- net SPARE_P226: now reaches J1.226 (P226)
- net SPARE_P226: now also J33.11 (Pin_11)
- net SPARE_P227: now reaches J1.227 (P227)
- net SPARE_P227: now also J33.12 (Pin_12)
- net SPARE_P228: now reaches J1.228 (P228)
- net SPARE_P228: now also J33.13 (Pin_13)
- net SPARE_P229: now reaches J1.229 (P229)
- net SPARE_P229: now also J33.14 (Pin_14)
- net SPARE_P230: now reaches J1.230 (P230)
- net SPARE_P230: now also J33.15 (Pin_15)
- net SPARE_P231: now reaches J1.231 (P231)
- net SPARE_P231: now also J33.16 (Pin_16)
- net SPARE_P232: now reaches J1.232 (P232)
- net SPARE_P232: now also J33.17 (Pin_17)
- net SPARE_P233: now reaches J1.233 (P233)
- net SPARE_P233: now also J33.18 (Pin_18)
- net SPARE_P234: now reaches J1.234 (P234)
- net SPARE_P234: now also J33.19 (Pin_19)
- net SPARE_P235: now reaches J1.235 (P235)
- net SPARE_P235: now also J33.20 (Pin_20)
- net SPARE_P236: now reaches J1.236 (P236)
- net SPARE_P236: now also J33.21 (Pin_21)
- net SPARE_P237: now reaches J1.237 (P237)
- net SPARE_P237: now also J33.22 (Pin_22)
- net SPARE_P238: now reaches J1.238 (P238)
- net SPARE_P238: now also J33.23 (Pin_23)
- net SPARE_P239: now reaches J1.239 (P239)
- net SPARE_P239: now also J33.24 (Pin_24)
- net SPARE_P240: now reaches J1.240 (P240)
- net SPARE_P240: now also J33.25 (Pin_25)
- net SAR_AUX0: now reaches J1.146 (P146)
- net SAR_AUX0: now also J28.2 (Pin_2)
- net SMB0_SDA: now reaches J1.148 (P148)
- net SMB0_SDA: now also J29.2 (Pin_2)
- net SMB0_SCK: now reaches J1.149 (P149)
- net SMB0_SCK: now also J29.3 (Pin_3)
- net SMB1_SDA: now reaches J1.150 (P150)
- net SMB1_SDA: now also J29.4 (Pin_4)
- net SMB1_SCK: now reaches J1.151 (P151)
- net SMB1_SCK: now also J29.5 (Pin_5)
- net GPIO0: now reaches J1.153 (P153)
- net GPIO0: now also J30.2 (Pin_2)
- net GPIO1: now reaches J1.154 (P154)
- net GPIO1: now also J30.3 (Pin_3)
- net GPIO2: now reaches J1.155 (P155)
- net GPIO2: now also J30.4 (Pin_4)
- net GPIO3: now reaches J1.156 (P156)
- net GPIO3: now also J30.5 (Pin_5)
- net GPIO4: now reaches J1.157 (P157)
- net GPIO4: now also J30.6 (Pin_6)
- net GPIO5: now reaches J1.158 (P158)
- net GPIO5: now also J30.7 (Pin_7)
- net GPIO6: now reaches J1.159 (P159)
- net GPIO6: now also J30.8 (Pin_8)
- net GPIO7: now reaches J1.160 (P160)
- net GPIO7: now also J30.9 (Pin_9)
- net GPIO8: now reaches J1.161 (P161)
- net GPIO8: now also J30.10 (Pin_10)
- net GPIO9: now reaches J1.162 (P162)
- net GPIO9: now also J30.11 (Pin_11)
- net GPIO10: now reaches J1.163 (P163)
- net GPIO10: now also J30.12 (Pin_12)
- net GPIO11: now reaches J1.164 (P164)
- net GPIO11: now also J30.13 (Pin_13)
- net GPIO12: now reaches J1.165 (P165)
- net GPIO12: now also J30.14 (Pin_14)
- net GPIO13: now reaches J1.166 (P166)
- net GPIO13: now also J30.15 (Pin_15)
- net GPIO14: now reaches J1.167 (P167)
- net GPIO14: now also J30.16 (Pin_16)
- net GPIO15: now reaches J1.168 (P168)
- net GPIO15: now also J30.17 (Pin_17)
- net SPARE_P170: now reaches J1.170 (P170)
- net SPARE_P170: now also J31.2 (Pin_2)
- net SPARE_P171: now reaches J1.171 (P171)
- net SPARE_P171: now also J31.3 (Pin_3)
- net SPARE_P172: now reaches J1.172 (P172)
- net SPARE_P172: now also J31.4 (Pin_4)
- net SPARE_P173: now reaches J1.173 (P173)
- net SPARE_P173: now also J31.5 (Pin_5)
- net SPARE_P174: now reaches J1.174 (P174)
- net SPARE_P174: now also J31.6 (Pin_6)
- net SPARE_P175: now reaches J1.175 (P175)
- net SPARE_P175: now also J31.7 (Pin_7)
- net SPARE_P176: now reaches J1.176 (P176)
- net SPARE_P176: now also J31.8 (Pin_8)
- net SPARE_P177: now reaches J1.177 (P177)
- net SPARE_P177: now also J31.9 (Pin_9)
- net SPARE_P178: now reaches J1.178 (P178)
- net SPARE_P178: now also J31.10 (Pin_10)
- net SPARE_P179: now reaches J1.179 (P179)
- net SPARE_P179: now also J31.11 (Pin_11)
- net SPARE_P180: now reaches J1.180 (P180)
- net SPARE_P180: now also J31.12 (Pin_12)
- net SPARE_P181: now reaches J1.181 (P181)
- net SPARE_P181: now also J31.13 (Pin_13)
- net SPARE_P182: now reaches J1.182 (P182)
- net SPARE_P182: now also J31.14 (Pin_14)
- net SPARE_P183: now reaches J1.183 (P183)
- net SPARE_P183: now also J31.15 (Pin_15)
- net SPARE_P184: now reaches J1.184 (P184)
- net SPARE_P184: now also J31.16 (Pin_16)
- net SPARE_P185: now reaches J1.185 (P185)
- net SPARE_P185: now also J31.17 (Pin_17)
- net SPARE_P186: now reaches J1.186 (P186)
- net SPARE_P186: now also J31.18 (Pin_18)
- net SPARE_P187: now reaches J1.187 (P187)
- net SPARE_P187: now also J31.19 (Pin_19)
- net SPARE_P188: now reaches J1.188 (P188)
- net SPARE_P188: now also J31.20 (Pin_20)
- net SPARE_P189: now reaches J1.189 (P189)
- net SPARE_P189: now also J31.21 (Pin_21)
- net SPARE_P190: now reaches J1.190 (P190)
- net SPARE_P190: now also J31.22 (Pin_22)
- net SPARE_P191: now reaches J1.191 (P191)
- net SPARE_P191: now also J31.23 (Pin_23)
- net SPARE_P192: now reaches J1.192 (P192)
- net SPARE_P192: now also J31.24 (Pin_24)
- net SPARE_P241: now reaches J1.241 (P241)
- net SPARE_P241: now also J34.2 (Pin_2)
- net SPARE_P242: now reaches J1.242 (P242)
- net SPARE_P242: now also J34.3 (Pin_3)
- net SPARE_P243: now reaches J1.243 (P243)
- net SPARE_P243: now also J34.4 (Pin_4)
- net SPARE_P244: now reaches J1.244 (P244)
- net SPARE_P244: now also J34.5 (Pin_5)
- net SPARE_P245: now reaches J1.245 (P245)
- net SPARE_P245: now also J34.6 (Pin_6)
- net SPARE_P246: now reaches J1.246 (P246)
- net SPARE_P246: now also J34.7 (Pin_7)
- net SPARE_P247: now reaches J1.247 (P247)
- net SPARE_P247: now also J34.8 (Pin_8)
- net SPARE_P248: now reaches J1.248 (P248)
- net SPARE_P248: now also J34.9 (Pin_9)
- net SPARE_P249: now reaches J1.249 (P249)
- net SPARE_P249: now also J34.10 (Pin_10)
- net SPARE_P250: now reaches J1.250 (P250)
- net SPARE_P250: now also J34.11 (Pin_11)
- net SPARE_P251: now reaches J1.251 (P251)
- net SPARE_P251: now also J34.12 (Pin_12)
- net SPARE_P252: now reaches J1.252 (P252)
- net SPARE_P252: now also J34.13 (Pin_13)
- net SPARE_P253: now reaches J1.253 (P253)
- net SPARE_P253: now also J34.14 (Pin_14)
- net SPARE_P254: now reaches J1.254 (P254)
- net SPARE_P254: now also J34.15 (Pin_15)
- net SPARE_P255: now reaches J1.255 (P255)
- net SPARE_P255: now also J34.16 (Pin_16)
- net SPARE_P256: now reaches J1.256 (P256)
- net SPARE_P256: now also J34.17 (Pin_17)
- net SPARE_P257: now reaches J1.257 (P257)
- net SPARE_P257: now also J34.18 (Pin_18)
- net SPARE_P258: now reaches J1.258 (P258)
- net SPARE_P258: now also J34.19 (Pin_19)
- net SPARE_P259: now reaches J1.259 (P259)
- net SPARE_P259: now also J34.20 (Pin_20)
- net SPARE_P260: now reaches J1.260 (P260)
- net SPARE_P260: now also J34.21 (Pin_21)
- net SPARE_P261: now reaches J1.261 (P261)
- net SPARE_P261: now also J34.22 (Pin_22)
- net SPARE_P262: now reaches J1.262 (P262)
- net SPARE_P262: now also J34.23 (Pin_23)
- net SPARE_P263: now reaches J1.263 (P263)
- net SPARE_P263: now also J34.24 (Pin_24)
- net SPARE_P264: now reaches J1.264 (P264)
- net SPARE_P264: now also J34.25 (Pin_25)
- net SPARE_P265: now reaches J1.265 (P265)
- net SPARE_P265: now also J35.2 (Pin_2)
- net SPARE_P266: now reaches J1.266 (P266)
- net SPARE_P266: now also J35.3 (Pin_3)
- net SPARE_P267: now reaches J1.267 (P267)
- net SPARE_P267: now also J35.4 (Pin_4)
- net SPARE_P268: now reaches J1.268 (P268)
- net SPARE_P268: now also J35.5 (Pin_5)
- net SPARE_P269: now reaches J1.269 (P269)
- net SPARE_P269: now also J35.6 (Pin_6)
- net SPARE_P270: now reaches J1.270 (P270)
- net SPARE_P270: now also J35.7 (Pin_7)
- net SPARE_P271: now reaches J1.271 (P271)
- net SPARE_P271: now also J35.8 (Pin_8)
- net SPARE_P272: now reaches J1.272 (P272)
- net SPARE_P272: now also J35.9 (Pin_9)
- net SPARE_P273: now reaches J1.273 (P273)
- net SPARE_P273: now also J35.10 (Pin_10)
- net SPARE_P274: now reaches J1.274 (P274)
- net SPARE_P274: now also J35.11 (Pin_11)
- net SPARE_P275: now reaches J1.275 (P275)
- net SPARE_P275: now also J35.12 (Pin_12)
- net SPARE_P276: now reaches J1.276 (P276)
- net SPARE_P276: now also J35.13 (Pin_13)
- net SPARE_P277: now reaches J1.277 (P277)
- net SPARE_P277: now also J35.14 (Pin_14)
- net SPARE_P278: now reaches J1.278 (P278)
- net SPARE_P278: now also J35.15 (Pin_15)
- net SPARE_P279: now reaches J1.279 (P279)
- net SPARE_P279: now also J35.16 (Pin_16)
- net SPARE_P280: now reaches J1.280 (P280)
- net SPARE_P280: now also J35.17 (Pin_17)
- net SPARE_P281: now reaches J1.281 (P281)
- net SPARE_P281: now also J35.18 (Pin_18)
- net SPARE_P282: now reaches J1.282 (P282)
- net SPARE_P282: now also J35.19 (Pin_19)
- net SPARE_P283: now reaches J1.283 (P283)
- net SPARE_P283: now also J35.20 (Pin_20)
- net SPARE_P284: now reaches J1.284 (P284)
- net SPARE_P284: now also J35.21 (Pin_21)
- net SPARE_P285: now reaches J1.285 (P285)
- net SPARE_P285: now also J35.22 (Pin_22)
- net SPARE_P286: now reaches J1.286 (P286)
- net SPARE_P286: now also J35.23 (Pin_23)
- net SPARE_P287: now reaches J1.287 (P287)
- net SPARE_P287: now also J35.24 (Pin_24)
- net SPARE_P288: now reaches J1.288 (P288)
- net SPARE_P288: now also J35.25 (Pin_25)
- net UART0_CTS: now reaches J1.100 (P100)
- net UART0_CTS: now also J22.4 (Pin_4)
- net UART0_RTS: now reaches J1.101 (P101)
- net UART0_RTS: now also J22.5 (Pin_5)
- net UART2_RXD: now reaches J1.103 (P103)
- net UART2_RXD: now also J23.2 (Pin_2)
- net UART2_TXD: now reaches J1.104 (P104)
- net UART2_TXD: now also J23.3 (Pin_3)
- net UART2_CTS: now reaches J1.105 (P105)
- net UART2_CTS: now also J23.4 (Pin_4)
- net UART2_RTS: now reaches J1.106 (P106)
- net UART2_RTS: now also J23.5 (Pin_5)
- net UART3_RXD: now reaches J1.108 (P108)
- net UART3_RXD: now also J24.2 (Pin_2)
- net UART3_TXD: now reaches J1.109 (P109)
- net UART3_TXD: now also J24.3 (Pin_3)
- net UART3_CTS: now reaches J1.110 (P110)
- net UART3_CTS: now also J24.4 (Pin_4)
- net UART3_RTS: now reaches J1.111 (P111)
- net UART3_RTS: now also J24.5 (Pin_5)
- net GMAC1_MDIO: now reaches J1.113 (P113)
- net GMAC1_MDIO: now also J21.2 (Pin_2)
- net GMAC1_MDCK: now reaches J1.114 (P114)
- net GMAC1_MDCK: now also J21.3 (Pin_3)
- net GMAC1_TXCLK: now reaches J1.115 (P115)
- net GMAC1_TXCLK: now also J21.4 (Pin_4)
- net GMAC1_PHYCLK: now reaches J1.116 (P116)
- net GMAC1_PHYCLK: now also J21.5 (Pin_5)
- net GMAC1_TXEN: now reaches J1.117 (P117)
- net GMAC1_TXEN: now also J21.6 (Pin_6)
- net GMAC1_TXD0: now reaches J1.118 (P118)
- net GMAC1_TXD0: now also J21.7 (Pin_7)
- net GMAC1_TXD1: now reaches J1.119 (P119)
- net GMAC1_TXD1: now also J21.8 (Pin_8)
- net GMAC1_RXDV: now reaches J1.120 (P120)
- net GMAC1_RXDV: now also J21.9 (Pin_9)
- net GMAC1_RXD0: now reaches J1.121 (P121)
- net GMAC1_RXD0: now also J21.10 (Pin_10)
- net GMAC1_RXD1: now reaches J1.122 (P122)
- net GMAC1_RXD1: now also J21.11 (Pin_11)
- net SSI0_CLK: now reaches J1.124 (P124)
- net SSI0_CLK: now also J25.2 (Pin_2)
- net SSI0_DT: now reaches J1.125 (P125)
- net SSI0_DT: now also J25.3 (Pin_3)
- net SSI0_DR: now reaches J1.126 (P126)
- net SSI0_DR: now also J25.4 (Pin_4)
- net SSI0_CE0: now reaches J1.127 (P127)
- net SSI0_CE0: now also J25.5 (Pin_5)
- net SSI0_CE1: now reaches J1.128 (P128)
- net SSI0_CE1: now also J25.6 (Pin_6)
- net SSI0_GPC: now reaches J1.129 (P129)
- net SSI0_GPC: now also J25.7 (Pin_7)
- net SSI1_CLK: now reaches J1.131 (P131)
- net SSI1_CLK: now also J26.2 (Pin_2)
- net SSI1_DT: now reaches J1.132 (P132)
- net SSI1_DT: now also J26.3 (Pin_3)
- net SSI1_DR: now reaches J1.133 (P133)
- net SSI1_DR: now also J26.4 (Pin_4)
- net SSI1_CE0: now reaches J1.134 (P134)
- net SSI1_CE0: now also J26.5 (Pin_5)
- net PWM0: now reaches J1.136 (P136)
- net PWM0: now also J27.2 (Pin_2)
- net PWM1: now reaches J1.137 (P137)
- net PWM1: now also J27.3 (Pin_3)
- net PWM2: now reaches J1.138 (P138)
- net PWM2: now also J27.4 (Pin_4)
- net PWM3: now reaches J1.139 (P139)
- net PWM3: now also J27.5 (Pin_5)
- net PWM4: now reaches J1.140 (P140)
- net PWM4: now also J27.6 (Pin_6)
- net PWM5: now reaches J1.141 (P141)
- net PWM5: now also J27.7 (Pin_7)
- net PWM6: now reaches J1.142 (P142)
- net PWM6: now also J27.8 (Pin_8)
- net PWM7: now reaches J1.143 (P143)
- net PWM7: now also J27.9 (Pin_9)
- net UART0_RXD: now reaches J1.98 (P98)
- net UART0_RXD: now also J22.2 (Pin_2)
- net UART0_TXD: now reaches J1.99 (P99)
- net UART0_TXD: now also J22.3 (Pin_3)
- net RESERVED_P87 renamed GMAC0_MDIO
- net GMAC0_MDIO: now also J20.2 (Pin_2)
- net RESERVED_P88 renamed GMAC0_MDCK
- net GMAC0_MDCK: now also J20.3 (Pin_3)
- net RESERVED_P89 renamed GMAC0_TXCLK
- net GMAC0_TXCLK: now also J20.4 (Pin_4)
- net RESERVED_P90 renamed GMAC0_PHYCLK
- net GMAC0_PHYCLK: now also J20.5 (Pin_5)
- net RESERVED_P91 renamed GMAC0_TXEN
- net GMAC0_TXEN: now also J20.6 (Pin_6)
- net RESERVED_P92 renamed GMAC0_TXD0
- net GMAC0_TXD0: now also J20.7 (Pin_7)
- net RESERVED_P93 renamed GMAC0_TXD1
- net GMAC0_TXD1: now also J20.8 (Pin_8)
- net RESERVED_P94 renamed GMAC0_RXDV
- net GMAC0_RXDV: now also J20.9 (Pin_9)
- net RESERVED_P95 renamed GMAC0_RXD0
- net GMAC0_RXD0: now also J20.10 (Pin_10)
- net RESERVED_P96 renamed GMAC0_RXD1
- net GMAC0_RXD1: now also J20.11 (Pin_11)
- net VCORE_FB renamed VCORE_FB_DIGIPOT
- net VCORE_FB_DIGIPOT: now also JP6.2 (Pin_2); no longer U1.12 (FB)
- net VDDR_FB renamed VDDR_FB_DIGIPOT
- net VDDR_FB_DIGIPOT: now also JP10.2 (Pin_2); no longer U2.4 (FB)
- new net VCORE_FB_0V8: JP2.2 (Pin_2), R27.2, R28.1
- new net VCORE_FB_0V9: JP3.2 (Pin_2), R29.2, R30.1
- new net VCORE_FB_1V0: JP4.2 (Pin_2), R31.2, R32.1
- new net VCORE_FB_1V1: JP5.2 (Pin_2), R33.2, R34.1
- new net VCORE_FB_SEL: JP2.1 (Pin_1), JP3.1 (Pin_1), JP4.1 (Pin_1), JP5.1 (Pin_1), JP6.1 (Pin_1), U1.12 (FB)
- new net VDDR_FB_1V35: JP7.2 (Pin_2), R35.2, R36.1
- new net VDDR_FB_1V5: JP8.2 (Pin_2), R37.2, R38.1
- new net VDDR_FB_1V8: JP9.2 (Pin_2), R39.2, R40.1
- new net VDDR_FB_SEL: JP10.1 (Pin_1), JP7.1 (Pin_1), JP8.1 (Pin_1), JP9.1 (Pin_1), U2.4 (FB)
Other:
- note added: "GMAC0 (RGMII0)"
- note added: "GMAC1 (RGMII1, A1 2nd MAC)"
- note added: "GPIO0-15 (plain)"
- note added: "J1 SPARE (P170-192)"
- note added: "J1 SPARE (P193-216)"
- note added: "J1 SPARE (P217-240)"
- note added: "J1 SPARE (P241-264)"
- note added: "J1 SPARE (P265-288)"
- note added: "PIN BREAKOUT HEADERS"
- note added: "PWM0-7"
- note added: "SAR-ADC"
- note added: "SMB0/SMB1 (general I2C)"
- note added: "SSI0 (SPI master)"
- note added: "SSI1"
- note added: "UART0"
- note added: "UART2"
- note added: "UART3"
- note added: "VCORE VOLTAGE SELECT"
- note added: "VDDR VOLTAGE SELECT"

Commit message: Fix schematic<->PCB linking, reorder J1 pins by connected peer, add +3V3 plane, wire microSD card-detect
- schgen.py: deterministic per-symbol UUIDs (uuid5, keyed on ref designator)
  instead of random uuid4, so PCB footprints stay linked to their schematic
  symbol across regenerations; link all 133 real PCB footprints to their
  schematic symbol via path, fixing "Update PCB from Schematic" placing
  duplicates.
- J1 pin reorg: audio (HPOUTL/MICLP) moved from 170/171 to 6/7 (170/171 now
  GND); USBA_HOST_DP/DM moved from 40/41 to 20/21 (40/41 now GND); the 20
  pins connected directly to U8 (ESP32-S3) reordered so U8's ascending pin
  number maps to J1's descending pin number; +5V_MODEA (redundant -- a
  self-contained module already needs its own bare-bench power input)
  replaced with +5V_SW (the real arbitrated switched-5V rail) on pins 17/18.
- New +3V3 copper pour on In1.Cu, mirroring the existing GND pour; every
  +3V3 pad on the board (38, now 39 with R43) gets a stub trace + via down
  to it.
- microSD (J4): switched to the Micro_SD_Card_Det2 symbol so pin 10 (the
  footprint's real card-detect pad) has somewhere to attach; added R43
  (1M, matches TeaCup 3.3's R22) pulling MSC0_CD up to +3V3.
- fp-lib-table: replaced hardcoded /usr/share/kicad/footprints/... paths
  with ${KICAD10_FOOTPRINT_DIR}, fixing "footprint not found" errors for
  every component when Update PCB from Schematic runs outside this Linux
  environment.

Verified throughout via isolated ERC/DRC diffs against pre-change
baselines; each change confirmed to produce only its own intended delta.
Parts:
- removed J20: HDR_J20, Connector_PinHeader_2.54mm:PinHeader_1x11_P2.54mm_Vertical, symbol Connector_Generic:Conn_01x11
- removed J21: HDR_J21, Connector_PinHeader_2.54mm:PinHeader_1x11_P2.54mm_Vertical, symbol Connector_Generic:Conn_01x11
- removed J25: HDR_J25, Connector_PinHeader_2.54mm:PinHeader_1x07_P2.54mm_Vertical, symbol Connector_Generic:Conn_01x07
- removed J27: HDR_J27, Connector_PinHeader_2.54mm:PinHeader_1x09_P2.54mm_Vertical, symbol Connector_Generic:Conn_01x09
- removed J30: HDR_J30, Connector_PinHeader_2.54mm:PinHeader_1x17_P2.54mm_Vertical, symbol Connector_Generic:Conn_01x17
- removed J31: HDR_J31, Connector_PinHeader_2.54mm:PinHeader_1x24_P2.54mm_Vertical, symbol Connector_Generic:Conn_01x24
- removed J32: HDR_J32, Connector_PinHeader_2.54mm:PinHeader_1x25_P2.54mm_Vertical, symbol Connector_Generic:Conn_01x25
- removed J33: HDR_J33, Connector_PinHeader_2.54mm:PinHeader_1x25_P2.54mm_Vertical, symbol Connector_Generic:Conn_01x25
- removed J34: HDR_J34, Connector_PinHeader_2.54mm:PinHeader_1x25_P2.54mm_Vertical, symbol Connector_Generic:Conn_01x25
- removed J35: HDR_J35, Connector_PinHeader_2.54mm:PinHeader_1x25_P2.54mm_Vertical, symbol Connector_Generic:Conn_01x25
- removed J4: Hirose_DM3D-SF, Connector_Card:microSD_HC_Hirose_DM3D-SF, symbol Connector:Micro_SD_Card
- removed Q1, Q2: AO3401A, Package_TO_SOT_SMD:SOT-23, symbol Device:Q_PMOS
- added J20: HDR_J20, Connector_PinHeader_2.54mm:PinHeader_2x06_P2.54mm_Vertical, symbol Connector_Generic:Conn_02x06_Odd_Even
- added J21: HDR_J21, Connector_PinHeader_2.54mm:PinHeader_2x06_P2.54mm_Vertical, symbol Connector_Generic:Conn_02x06_Odd_Even
- added J25: HDR_J25, Connector_PinHeader_2.54mm:PinHeader_2x04_P2.54mm_Vertical, symbol Connector_Generic:Conn_02x04_Odd_Even
- added J27: HDR_J27, Connector_PinHeader_2.54mm:PinHeader_2x05_P2.54mm_Vertical, symbol Connector_Generic:Conn_02x05_Odd_Even
- added J30: HDR_J30, Connector_PinHeader_2.54mm:PinHeader_2x09_P2.54mm_Vertical, symbol Connector_Generic:Conn_02x09_Odd_Even
- added J31: HDR_J31, Connector_PinHeader_2.54mm:PinHeader_2x11_P2.54mm_Vertical, symbol Connector_Generic:Conn_02x11_Odd_Even
- added J32: HDR_J32, Connector_PinHeader_2.54mm:PinHeader_2x13_P2.54mm_Vertical, symbol Connector_Generic:Conn_02x13_Odd_Even
- added J33: HDR_J33, Connector_PinHeader_2.54mm:PinHeader_2x13_P2.54mm_Vertical, symbol Connector_Generic:Conn_02x13_Odd_Even
- added J34: HDR_J34, Connector_PinHeader_2.54mm:PinHeader_2x13_P2.54mm_Vertical, symbol Connector_Generic:Conn_02x13_Odd_Even
- added J35: HDR_J35, Connector_PinHeader_2.54mm:PinHeader_2x13_P2.54mm_Vertical, symbol Connector_Generic:Conn_02x13_Odd_Even
- added J36: HDR_J36, Connector_PinHeader_2.54mm:PinHeader_1x03_P2.54mm_Vertical, symbol Connector_Generic:Conn_01x03
- added J37: HDR_J37, Connector_PinHeader_2.54mm:PinHeader_1x07_P2.54mm_Vertical, symbol Connector_Generic:Conn_01x07
- added J38: AMP_MIC_TAP, Connector_PinHeader_2.54mm:PinHeader_1x03_P2.54mm_Vertical, symbol Connector_Generic:Conn_01x03
- added J4: Hirose_DM3D-SF, Connector_Card:microSD_HC_Hirose_DM3D-SF, symbol Connector:Micro_SD_Card_Det2
- added JP11, JP12: EN_SEL, Connector_PinHeader_2.54mm:PinHeader_1x03_P2.54mm_Vertical_SMD_Pin1Left, symbol Connector_Generic:Conn_01x03
- added Q1, Q2: AO3401A, Package_TO_SOT_SMD:SOT-23, symbol Transistor_FET:AO3401A
- added R43: 1M, Resistor_SMD:R_0402_1005Metric, symbol Device:R
- C13, C23: value 1nF_TBD -> 1nF
- D1, D2: footprint Diode_SMD:D_SOD-123W -> Diode_SMD:Nexperia_CFP3_SOD-123W
- U13: footprint Package_SO:SOIC-8_5.23x5.23mm_P1.27mm -> Package_SO:SOIC-8_5.3x5.3mm_P1.27mm
Connections:
- net +5V_MODEA is gone; now on net +5V_SW: J1.17 (P17), J1.18 (P18)
- net SPARE_P170 is gone; now on net GND: J1.170 (P170)
- net SPARE_P171 is gone; now on net GND: J1.171 (P171)
- net SPARE_P172 is gone; now on net GND: J1.172 (P172)
- net +3V3: now also J7.1, J7.4, J8.1, J8.4, J4.4 (VDD), JP11.3 (Pin_3), JP12.3 (Pin_3), R43.1; no longer J7.5, J8.5
- net +5V_ALT: now also Q1.3 (D), Q2.3 (D)
- net ALTUSB_VBUS: now also Q2.2 (S)
- net BOOTSEL: now also J1.35 (P35); no longer J1.26 (P26)
- net DCJACK_VBUS: now also Q1.2 (S)
- net EN_SW_ALT: now also SW2.1; no longer SW2.4
- net EN_SW_BMC: now also SW2.4; no longer SW2.1
- net GMAC0_MDCK: now also J20.3 (Pin_3)
- net GMAC0_MDIO: now also J20.2 (Pin_2)
- net GMAC0_PHYCLK: now also J20.5 (Pin_5)
- net GMAC0_RXD0: now also J20.10 (Pin_10)
- net GMAC0_RXD1: now also J20.11 (Pin_11)
- net GMAC0_RXDV: now also J20.9 (Pin_9)
- net GMAC0_TXCLK: now also J20.4 (Pin_4)
- net GMAC0_TXD0: now also J20.7 (Pin_7)
- net GMAC0_TXD1: now also J20.8 (Pin_8)
- net GMAC0_TXEN: now also J20.6 (Pin_6)
- net GMAC1_MDCK: now also J21.3 (Pin_3)
- net GMAC1_MDIO: now also J21.2 (Pin_2)
- net GMAC1_PHYCLK: now also J21.5 (Pin_5)
- net GMAC1_RXD0: now also J21.10 (Pin_10)
- net GMAC1_RXD1: now also J21.11 (Pin_11)
- net GMAC1_RXDV: now also J21.9 (Pin_9)
- net GMAC1_TXCLK: now also J21.4 (Pin_4)
- net GMAC1_TXD0: now also J21.7 (Pin_7)
- net GMAC1_TXD1: now also J21.8 (Pin_8)
- net GMAC1_TXEN: now also J21.6 (Pin_6)
- net GND: now also J1.41 (P41), J1.58 (P58), J1.86 (P86), J6.R2, J20.1 (Pin_1), J20.12 (Pin_12), J21.1 (Pin_1), J21.12 (Pin_12), J25.1 (Pin_1), J25.8 (Pin_8), J27.1 (Pin_1), J27.10 (Pin_10), J30.1 (Pin_1), J30.18 (Pin_18), J31.1 (Pin_1), J31.22 (Pin_22), J32.1 (Pin_1), J32.26 (Pin_26), J33.1 (Pin_1), J33.26 (Pin_26), J34.1 (Pin_1), J34.26 (Pin_26), J35.1 (Pin_1), J35.20 (Pin_20), J35.21 (Pin_21), J35.22 (Pin_22), J35.23 (Pin_23), J35.24 (Pin_24), J35.25 (Pin_25), J35.26 (Pin_26), J36.1 (Pin_1), J37.1 (Pin_1), J38.2 (Pin_2), J4.6 (VSS), J4.9 (DET_B); no longer J1.20 (P20), J1.21 (P21), J1.6 (P6), J1.7 (P7), J6.G, J7.1, J8.1
- net GPIO0: now also J30.2 (Pin_2)
- net GPIO1: now also J30.3 (Pin_3)
- net GPIO10: now also J30.12 (Pin_12)
- net GPIO11: now also J30.13 (Pin_13)
- net GPIO12: now also J30.14 (Pin_14)
- net GPIO13: now also J30.15 (Pin_15)
- net GPIO14: now also J30.16 (Pin_16)
- net GPIO15: now also J30.17 (Pin_17)
- net GPIO2: now also J30.4 (Pin_4)
- net GPIO3: now also J30.5 (Pin_5)
- net GPIO4: now also J30.6 (Pin_6)
- net GPIO5: now also J30.7 (Pin_7)
- net GPIO6: now also J30.8 (Pin_8)
- net GPIO7: now also J30.9 (Pin_9)
- net GPIO8: now also J30.10 (Pin_10)
- net GPIO9: now also J30.11 (Pin_11)
- net HOSTED_DATA_READY: now also J1.24 (P24); no longer J1.48 (P48)
- net HOSTED_HANDSHAKE: now also J1.25 (P25); no longer J1.47 (P47)
- net HOSTED_RESET: now also J1.48 (P48); no longer J1.86 (P86)
- net HOSTED_SPI_CLK: now also J1.45 (P45); no longer J1.43 (P43)
- net HOSTED_SPI_CS: now also J1.26 (P26); no longer J1.46 (P46)
- net HOSTED_SPI_MISO: now also J1.27 (P27); no longer J1.45 (P45)
- net HPOUTL: now also J1.7 (P7), J6.R1, J38.1 (Pin_1); no longer J1.58 (P58)
- net I2C_ID_SCL: now also J1.46 (P46); no longer J1.24 (P24)
- net I2C_ID_SDA: now also J1.47 (P47); no longer J1.23 (P23)
- net MIPI0_CLKN: now also J1.65 (P65), J7.8; no longer J1.70 (P70), J7.13
- net MIPI0_CLKP: now also J1.64 (P64), J7.7; no longer J1.71 (P71), J7.14
- net MIPI0_D0N: now also J1.71 (P71), J7.14; no longer J1.64 (P64), J7.7
- net MIPI0_D0P: now also J1.70 (P70), J7.13; no longer J1.65 (P65), J7.8
- net MIPI0_D1N: now also J1.68 (P68), J7.11; no longer J1.67 (P67), J7.10
- net MIPI0_D1P: now also J1.67 (P67), J7.10; no longer J1.68 (P68), J7.11
- net MIPI0_GPIO: now also J1.62 (P62), JP11.1 (Pin_1); no longer J1.60 (P60), J7.2
- net MIPI0_SCCB_SCL: now also J1.61 (P61), J7.3; no longer J1.62 (P62), J7.4
- net MIPI0_SCCB_SDA: now also J1.60 (P60), J7.2; no longer J1.61 (P61), J7.3
- net MIPI1_CLKN: now also J1.78 (P78), J8.8; no longer J1.83 (P83), J8.13
- net MIPI1_CLKP: now also J1.77 (P77), J8.7; no longer J1.84 (P84), J8.14
- net MIPI1_D0N: now also J1.84 (P84), J8.14; no longer J1.77 (P77), J8.7
- net MIPI1_D0P: now also J1.83 (P83), J8.13; no longer J1.78 (P78), J8.8
- net MIPI1_D1N: now also J1.81 (P81), J8.11; no longer J1.80 (P80), J8.10
- net MIPI1_D1P: now also J1.80 (P80), J8.10; no longer J1.81 (P81), J8.11
- net MIPI1_GPIO: now also J1.75 (P75), JP12.1 (Pin_1); no longer J1.73 (P73), J8.2
- net MIPI1_SCCB_SCL: now also J1.74 (P74), J8.3; no longer J1.75 (P75), J8.4
- net MIPI1_SCCB_SDA: now also J1.73 (P73), J8.2; no longer J1.74 (P74), J8.3
- net MSC0_CLK: now also J1.53 (P53), J4.5 (CLK); no longer J1.50 (P50)
- net MSC0_CMD: now also J1.54 (P54), J4.3 (CMD); no longer J1.52 (P52)
- net MSC0_D0: now also J1.52 (P52), J4.7 (DAT0); no longer J1.53 (P53)
- net MSC0_D1: now also J1.50 (P50), J4.8 (DAT1); no longer J1.54 (P54)
- net MSC0_D2: now also J1.56 (P56), J4.1 (DAT2); no longer J1.55 (P55)
- net MSC0_D3_CD: now also J1.55 (P55), J4.2 (DAT3/CD); no longer J1.56 (P56)
- net PWM0: now also J27.2 (Pin_2)
- net PWM1: now also J27.3 (Pin_3)
- net PWM2: now also J27.4 (Pin_4)
- net PWM3: now also J27.5 (Pin_5)
- net PWM4: now also J27.6 (Pin_6)
- net PWM5: now also J27.7 (Pin_7)
- net PWM6: now also J27.8 (Pin_8)
- net PWM7: now also J27.9 (Pin_9)
- net Q1_GATE: now also Q1.1 (G)
- net Q2_GATE: now also Q2.1 (G)
- net RESET_EN: now also J1.34 (P34); no longer J1.27 (P27)
- net SFC_CLK: now also J1.30 (P30); no longer J1.29 (P29)
- net SFC_CS: now also J1.32 (P32); no longer J1.28 (P28)
- net SFC_IO0: now also J1.31 (P31); no longer J1.30 (P30)
- net SFC_IO1: now also J1.29 (P29); no longer J1.31 (P31)
- net SFC_IO2: now also J1.28 (P28); no longer J1.32 (P32)
- net SPARE_P173: now also J31.2 (Pin_2)
- net SPARE_P174: now also J31.3 (Pin_3)
- net SPARE_P175: now also J31.4 (Pin_4)
- net SPARE_P176: now also J31.5 (Pin_5)
- net SPARE_P177: now also J31.6 (Pin_6)
- net SPARE_P178: now also J31.7 (Pin_7)
- net SPARE_P179: now also J31.8 (Pin_8)
- net SPARE_P180: now also J31.9 (Pin_9)
- net SPARE_P181: now also J31.10 (Pin_10)
- net SPARE_P182: now also J31.11 (Pin_11)
- net SPARE_P183: now also J31.12 (Pin_12)
- net SPARE_P184: now also J31.13 (Pin_13)
- net SPARE_P185: now also J31.14 (Pin_14)
- net SPARE_P186: now also J31.15 (Pin_15)
- net SPARE_P187: now also J31.16 (Pin_16)
- net SPARE_P188: now also J31.17 (Pin_17)
- net SPARE_P189: now also J31.18 (Pin_18)
- net SPARE_P190: now also J31.19 (Pin_19)
- net SPARE_P191: now also J31.20 (Pin_20)
- net SPARE_P192: now also J31.21 (Pin_21)
- net SPARE_P193: now also J32.2 (Pin_2)
- net SPARE_P194: now also J32.3 (Pin_3)
- net SPARE_P195: now also J32.4 (Pin_4)
- net SPARE_P196: now also J32.5 (Pin_5)
- net SPARE_P197: now also J32.6 (Pin_6)
- net SPARE_P198: now also J32.7 (Pin_7)
- net SPARE_P199: now also J32.8 (Pin_8)
- net SPARE_P200: now also J32.9 (Pin_9)
- net SPARE_P201: now also J32.10 (Pin_10)
- net SPARE_P202: now also J32.11 (Pin_11)
- net SPARE_P203: now also J32.12 (Pin_12)
- net SPARE_P204: now also J32.13 (Pin_13)
- net SPARE_P205: now also J32.14 (Pin_14)
- net SPARE_P206: now also J32.15 (Pin_15)
- net SPARE_P207: now also J32.16 (Pin_16)
- net SPARE_P208: now also J32.17 (Pin_17)
- net SPARE_P209: now also J32.18 (Pin_18)
- net SPARE_P210: now also J32.19 (Pin_19)
- net SPARE_P211: now also J32.20 (Pin_20)
- net SPARE_P212: now also J32.21 (Pin_21)
- net SPARE_P213: now also J32.22 (Pin_22)
- net SPARE_P214: now also J32.23 (Pin_23)
- net SPARE_P215: now also J32.24 (Pin_24)
- net SPARE_P216: now also J32.25 (Pin_25)
- net SPARE_P217: now also J33.2 (Pin_2)
- net SPARE_P218: now also J33.3 (Pin_3)
- net SPARE_P219: now also J33.4 (Pin_4)
- net SPARE_P220: now also J33.5 (Pin_5)
- net SPARE_P221: now also J33.6 (Pin_6)
- net SPARE_P222: now also J33.7 (Pin_7)
- net SPARE_P223: now also J33.8 (Pin_8)
- net SPARE_P224: now also J33.9 (Pin_9)
- net SPARE_P225: now also J33.10 (Pin_10)
- net SPARE_P226: now also J33.11 (Pin_11)
- net SPARE_P227: now also J33.12 (Pin_12)
- net SPARE_P228: now also J33.13 (Pin_13)
- net SPARE_P229: now also J33.14 (Pin_14)
- net SPARE_P230: now also J33.15 (Pin_15)
- net SPARE_P231: now also J33.16 (Pin_16)
- net SPARE_P232: now also J33.17 (Pin_17)
- net SPARE_P233: now also J33.18 (Pin_18)
- net SPARE_P234: now also J33.19 (Pin_19)
- net SPARE_P235: now also J33.20 (Pin_20)
- net SPARE_P236: now also J33.21 (Pin_21)
- net SPARE_P237: now also J33.22 (Pin_22)
- net SPARE_P238: now also J33.23 (Pin_23)
- net SPARE_P239: now also J33.24 (Pin_24)
- net SPARE_P240: now also J33.25 (Pin_25)
- net SPARE_P241: now also J34.2 (Pin_2)
- net SPARE_P242: now also J34.3 (Pin_3)
- net SPARE_P243: now also J34.4 (Pin_4)
- net SPARE_P244: now also J34.5 (Pin_5)
- net SPARE_P245: now also J34.6 (Pin_6)
- net SPARE_P246: now also J34.7 (Pin_7)
- net SPARE_P247: now also J34.8 (Pin_8)
- net SPARE_P248: now also J34.9 (Pin_9)
- net SPARE_P249: now also J34.10 (Pin_10)
- net SPARE_P250: now also J34.11 (Pin_11)
- net SPARE_P251: now also J34.12 (Pin_12)
- net SPARE_P252: now also J34.13 (Pin_13)
- net SPARE_P253: now also J34.14 (Pin_14)
- net SPARE_P254: now also J34.15 (Pin_15)
- net SPARE_P255: now also J34.16 (Pin_16)
- net SPARE_P256: now also J34.17 (Pin_17)
- net SPARE_P257: now also J34.18 (Pin_18)
- net SPARE_P258: now also J34.19 (Pin_19)
- net SPARE_P259: now also J34.20 (Pin_20)
- net SPARE_P260: now also J34.21 (Pin_21)
- net SPARE_P261: now also J34.22 (Pin_22)
- net SPARE_P262: now also J34.23 (Pin_23)
- net SPARE_P263: now also J34.24 (Pin_24)
- net SPARE_P264: now also J34.25 (Pin_25)
- net SPARE_P265: now also J35.2 (Pin_2)
- net SPARE_P266: now also J35.3 (Pin_3)
- net SPARE_P267: now also J35.4 (Pin_4)
- net SPARE_P268: now also J35.5 (Pin_5)
- net SPARE_P269: now also J35.6 (Pin_6)
- net SPARE_P270: now also J35.7 (Pin_7)
- net SPARE_P271: now also J35.8 (Pin_8)
- net SPARE_P272: now also J35.9 (Pin_9)
- net SPARE_P273: now also J35.10 (Pin_10)
- net SPARE_P274: now also J35.11 (Pin_11)
- net SPARE_P275: now also J35.12 (Pin_12)
- net SPARE_P276: now also J35.13 (Pin_13)
- net SPARE_P277: now also J35.14 (Pin_14)
- net SPARE_P278: now also J35.15 (Pin_15)
- net SPARE_P279: now also J35.16 (Pin_16)
- net SPARE_P280: now also J35.17 (Pin_17)
- net SPARE_P281: now also J35.18 (Pin_18)
- net SPARE_P282: now also J35.19 (Pin_19)
- net SSI0_CE0: now also J25.5 (Pin_5)
- net SSI0_CE1: now also J25.6 (Pin_6)
- net SSI0_CLK: now also J25.2 (Pin_2)
- net SSI0_DR: now also J25.4 (Pin_4)
- net SSI0_DT: now also J25.3 (Pin_3)
- net SSI0_GPC: now also J25.7 (Pin_7)
- net UART1_RX: now also J1.42 (P42), J36.2 (Pin_2); no longer J1.35 (P35)
- net UART1_TX: now also J1.43 (P43), J36.3 (Pin_3); no longer J1.34 (P34)
- net USBA_HOST_DM: now also J1.21 (P21); no longer J1.42 (P42)
- net USBA_HOST_DP: now also J1.20 (P20); no longer J1.41 (P41)
- net VCORE_SNS: now also J1.23 (P23); no longer J1.25 (P25)
- net MICLP: now reaches J6.S
- net MICLP: now also J1.6 (P6), J38.3 (Pin_3)
- net SPARE_P283 renamed MSC1_CLK
- net MSC1_CLK: now also J37.2 (Pin_2)
- net SPARE_P284 renamed MSC1_CMD
- net MSC1_CMD: now also J37.3 (Pin_3)
- net SPARE_P285 renamed MSC1_D0
- net MSC1_D0: now also J37.4 (Pin_4)
- net SPARE_P286 renamed MSC1_D1
- net MSC1_D1: now also J37.5 (Pin_5)
- net SPARE_P287 renamed MSC1_D2
- net MSC1_D2: now also J37.6 (Pin_6)
- net SPARE_P288 renamed MSC1_D3_CD
- net MSC1_D3_CD: now also J37.7 (Pin_7)
- new net MIPI0_SENSOR_EN: J7.5, JP11.2 (Pin_2)
- new net MIPI1_SENSOR_EN: J8.5, JP12.2 (Pin_2)
- new net MSC0_CD: J4.10 (DET_A), R43.2
Other:
- note added: "J1 SPARE (P173-192)"
- note added: "J1 SPARE (P265-282)"
- note added: "MSC1"
- note added: "UART1 (BMC console)"
- note removed: "J1 SPARE (P170-192)"
- note removed: "J1 SPARE (P265-288)"
