File: hw/interposer_t41/sheets/ddr4_edge.kicad_sch (KiCad schematic)
At the start: 1 part, among them J1 DIMM-DDR4

Commit message: Add T41 (QFN96) interposer board
Per-SoC interposer for the T41 QFN96 package, mirroring the T31ZX
interposer structure: SoC + fanout + clock + decoupling + straps on
a DDR4 UDIMM-288 card-edge, built with the same headless KiCad
pipeline (schgen.py / build_soc.py / build_pcb.py / merge_sheets.py).

Also picks up executable-bit changes on the T31ZX interposer files.
Parts:
- J1: footprint teacup-interposer:DIMM-DDR4 -> teacup-interposer-t41:DIMM-DDR4; symbol teacup-interposer:DIMM-DDR4 -> teacup-interposer-t41:DIMM-DDR4
Other:
- title: Teacup Universal - DDR4 UDIMM-288 Card Edge (interposer) -> Teacup Universal - DDR4 UDIMM-288 Card Edge (T41 interposer)
Changed lines of the file:
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@@
 	(paper "A2")
 	(title_block
-		(title "Teacup Universal - DDR4 UDIMM-288 Card Edge (interposer)")
+		(title "Teacup Universal - DDR4 UDIMM-288 Card Edge (T41 interposer)")
 		(date "2026-07-11")
 		(rev "A")
 		(company "Teacup Universal")
 	)
-	(symbol (lib_id "teacup-interposer:DIMM-DDR4") (at 101.6 508.0 0) (unit 1)
+	(symbol (lib_id "teacup-interposer-t41:DIMM-DDR4") (at 101.6 508.0 0) (unit 1)
 		(property "Reference" "J1" (at 101.6 311.15 0) (effects (font (size 1.27 1.27))))
 		(property "Value" "DIMM-DDR4" (at 101.6 704.85 0) (effects (font (size 1.27 1.27))))
-		(property "Footprint" "teacup-interposer:DIMM-DDR4" (at 101.6 508.0 0) (effects (font (size 1.27 1.27)) hide))
+		(property "Footprint" "teacup-interposer-t41:DIMM-DDR4" (at 101.6 508.0 0) (effects (font (size 1.27 1.27)) hide))
 	)
 	(symbol (lib_id "power:GND") (at 81.28 336.55 270) (unit 1)
@@
 		(property "Reference" "#DGND041" (at 121.92 394.97 0) (effects (font (size 1.27 1.27)) hide))
 		(property "Value" "GND" (at 127.0 394.97 270) (effects (font (size 1.27 1.27))))
+	)
+	(symbol (lib_id "power:PWR_FLAG") (at 76.2 495.3 0) (unit 1)
+		(property "Reference" "#PWR1" (at 76.2 492.3 0) (effects (font (size 1.27 1.27))))
+		(property "Value" "PWR_FLAG" (at 76.2 498.3 0) (effects (font (size 1.27 1.27))))
+	)
+	(symbol (lib_id "power:GND") (at 76.2 495.3 0) (unit 1)
+		(property "Reference" "#SGND042" (at 76.2 495.3 0) (effects (font (size 1.27 1.27)) hide))
+		(property "Value" "GND" (at 76.2 500.38 0) (effects (font (size 1.27 1.27))))
 	)
 	(global_label "VCORE" (at 81.28 326.39 180) (effects (font (size 1.27 1.27)) (justify right)))
@@
 	(global_label "MSC1_D3_CD" (at 121.92 689.61 0) (effects (font (size 1.27 1.27)) (justify left)))
 	(sheet_instances
-		(path "/d2e3f4a5-0001-4000-8000-000000000001"
-			(page "2")
+		(path "/f3a4b5c6-0001-4000-8000-000000000001"
+			(page "1")
 		)
 	)
