File: hw/interposer/teacup-interposer.kicad_sch (KiCad schematic)
At the start: 36 parts, among them IC1 T31ZX, J1 DIMM-DDR4, U4 W25Q32JVSS, Y1 24 MHz

Commit message: Backfill MPN/Manufacturer fields on carrier and interposer schematics
Placed symbol instances only carried Reference/Value/Footprint; MPN and
Manufacturer were never propagated from the library cache, so BOM export
had a blank MPN column for every part. Fills in MPN (and Manufacturer
where unambiguous) for the 32 parts whose Value string is already a real
manufacturer part number - ICs, diodes, MOSFETs, switches, and specific
connectors - across the carrier, T31ZX interposer, and T41 interposer.
Generic passives, headers, and jumpers are left untouched since their
Value is a spec, not a part number.

ERC-neutral: 426/175/169 violations before and after on the three files.
Parts:
- IC1: MPN (none) -> T31ZX; Manufacturer (none) -> Ingenic Semiconductor
- U4: MPN (none) -> W25Q32JVSS; Manufacturer (none) -> Winbond Electronics
Changed lines of the file:
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@@
 		(property "Value" "T31ZX" (at 177.8 292.1 0) (effects (font (size 1.27 1.27))))
 		(property "Footprint" "teacup-interposer:QFN35P900X900X90-89N-D" (at 177.8 203.2 0) (effects (font (size 1.27 1.27)) hide))
+		(property "MPN" "T31ZX" (at 177.8 203.2 0) (effects (font (size 1.27 1.27)) hide))
+		(property "Manufacturer" "Ingenic Semiconductor" (at 177.8 203.2 0) (effects (font (size 1.27 1.27)) hide))
 	)
 	(symbol (lib_id "power:GND") (at 280.67 147.32 180) (unit 1)
@@
 		(property "Value" "W25Q32JVSS" (at 88.9 64.77 0) (effects (font (size 1.27 1.27))))
 		(property "Footprint" "Package_SO:SOIC-8_5.3x5.3mm_P1.27mm" (at 88.9 57.15 0) (effects (font (size 1.27 1.27)) hide))
+		(property "MPN" "W25Q32JVSS" (at 88.9 57.15 0) (effects (font (size 1.27 1.27)) hide))
+		(property "Manufacturer" "Winbond Electronics" (at 88.9 57.15 0) (effects (font (size 1.27 1.27)) hide))
 	)
 	(symbol (lib_id "power:GND") (at 88.9 69.85 0) (unit 1)
