File: hw/interposer/teacup-interposer.kicad_sch (KiCad schematic)
At the start: 36 parts, among them IC1 T31ZX, J1 DIMM-DDR4, U4 W25Q32JVSS, Y1 24 MHz

Commit message: Carrier: S5 pull-ups, unused-pin test-pad breakouts, value-only silk
- Add R44-R49 (100k) pull-ups/pull-downs for the BMC<->SoC link, SFC_IO2/IO3 and NOR CE
- Break out unused U15 P11-P17, U8 SPIIO7/MTMS/console UART and U12 spare VBUS to 1.0mm test pads
- Tie J4 SHIELD and J6 G to GND; no-connect the remaining unused pins (ERC pin_not_connected 30 -> 0)
- Silkscreen: show values/part names instead of references for R/C/U/L/D/Q/SW/JP (J refs kept)
- Refill zones; remove stray no-net track segments
- Interposer: SFC shared-bus pinout/schematic updates
Parts:
- removed U4: W25Q32JVSS, Package_SO:SOIC-8_5.3x5.3mm_P1.27mm, symbol Memory_Flash:W25Q32JVSS
- added C47, C48, C49: 10uF, Capacitor_SMD:C_0603_1608Metric_Pad1.08x0.95mm_HandSolder, symbol Device:C
- added R22, R27, R28: 0R, Resistor_SMD:R_0402_1005Metric, symbol Device:R
- added R23, R24, R25, R26: 1k, Resistor_SMD:R_0402_1005Metric, symbol Device:R
Connections:
- net +1V8: now also C48.1
- net +3V3: now also C49.1
- net BOOTSEL: now also R24.1
- net GND: now also C47.2, C48.2, C49.2, R22.2
- net PWM0: now also R27.2
- net PWM1: now also R28.2
- net RESET_EN: now also R23.1
- net SFC_CLK: now also IC1.48 (SFC_CLK_PA27)
- net SFC_CS: now also IC1.45 (SFC_CE0_PA28)
- net SFC_IO0: now also IC1.47 (SFC_DT_PA23)
- net SFC_IO1: now also IC1.46 (SFC_DR_PA24)
- net SPARE_P173: now also R23.2
- net SPARE_P174: now also R22.1
- net SPARE_P179: now also R24.2
- net SPARE_P180: now also R26.2
- net SPARE_P181: now also R25.2
- net SSI0_CE0: no longer IC1.45 (SFC_CE0_PA28)
- net SSI0_CLK: no longer IC1.48 (SFC_CLK_PA27)
- net SSI0_DR: no longer IC1.46 (SFC_DR_PA24)
- net SSI0_DT: no longer IC1.47 (SFC_DT_PA23)
- net SSI1_DR: now also R28.1
- net SSI1_DT: now also R27.1
- net UART1_RX: now also R25.1
- net UART1_TX: now also R26.1
- net VCORE: now also C47.1
