File: hw/interposer/teacup-interposer.kicad_pcb (KiCad board)
At the start: 4 copper layers, 133.3 x 31.2 mm, 36 parts, among them IC1 T31ZX, J1 DIMM-DDR4, U4 W25Q32JVSS, Y1 24 MHz

Commit message: Fix MIPI netclass assignment and route MIPI0 differential pairs
- Fix netclass_patterns net-name mismatch that left all MIPI nets on
  Default instead of the MIPI class; assign all 18 MIPI0/MIPI1 nets
  (diff pairs + GPIO/SCCB control lines) to MIPI, trace_width 0.15mm
- Route the 6 MIPI0 differential pair nets (CLKP/N, D0P/N, D1P/N)
  between IC1 and J1, previously left unrouted
- Remove stale teacup-t41-B_Adhesive.gba gerber
Routing:
- net MSC1_CMD: track 96.1 -> 84.6 mm, vias 1 -> 2
- net MSC1_CLK: track 96.5 -> 86.6 mm, vias 1 -> 2
- net GND: track 87.6 -> 82.6 mm, vias 229 -> 227
- net MIPI0_CLKP: track 18.0 -> 21.8 mm
- net MIPI0_D1P: track 18.4 -> 21.9 mm
- net MIPI0_D1N: track 18.3 -> 21.4 mm
- net MIPI0_CLKN: track 19.6 -> 21.3 mm
- net USBA_HOST_DM: track 54.6 -> 56.3 mm, vias 2 -> 4
- net USBA_HOST_DP: track 54.5 -> 56.0 mm, vias 0 -> 2
- net MIPI0_D0P: track 20.7 -> 21.9 mm
- net +1V8: track 174.8 -> 174.3 mm

Commit message: Relink 5 orphaned footprints (R10, R11, C19, C21, U4)
Footprints had lost their library reference (empty Library:Name prefix),
confirmed against the TeaCup(C)3.3 reference netlist. Relinked via
KiCad's Change Footprint dialog, preserving position/rotation/nets.

DRC: schematic_parity 46->41, no new errors, 0 unconnected items.
Parts:
- C19: footprint C_0603_1608Metric -> Capacitor_SMD:C_0603_1608Metric
- C21: footprint C_0402_1005Metric -> Capacitor_SMD:C_0402_1005Metric
- R10, R11: footprint R_0603_1608Metric -> Resistor_SMD:R_0603_1608Metric
- U4: footprint SOIC-8_5.3x5.3mm_P1.27mm -> Package_SO:SOIC-8_5.3x5.3mm_P1.27mm
Changed lines of the file:
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@@
 		)
 	)
-	(footprint "R_0603_1608Metric"
+	(footprint "Resistor_SMD:R_0603_1608Metric"
 		(layer "F.Cu")
 		(at 165.18 89.53 180)
-		(descr "Resistor SMD 0603 (1608 Metric), square (rectangular) end terminal, IPC-7351 nominal, (Body size source: IPC-SM-782 page 72, https://www.pcb-3d.com/wordpress/wp-content/uploads/ipc-sm-782a_amendment_1_and_2.pdf), generated with kicad-footprint-generator")
+		(descr "Resistor SMD 0603 (1608 Metric), square (rectangular) end terminal, IPC-7351 nominal, (Body size source: IPC-SM-782 page 72, https://www.pcb-3d.com/wordpress/wp-content/uploads/ipc-sm-782a_amendment_1_and_2.pdf)")
 		(tags "resistor")
 		(property "Reference" "R10"
-			(at 0 -1.43 0)
+			(at 0 -1.43 180)
 			(layer "F.SilkS")
 			(effects
@@
 		)
 		(property "Value" "100k"
-			(at 0 1.43 0)
+			(at 0 1.43 180)
 			(layer "F.Fab")
 			(effects
@@
 		)
 		(property "Datasheet" ""
-			(at 0 0 0)
+			(at 0 0 180)
 			(layer "F.Fab")
 			(hide yes)
@@
 		)
 		(property "Description" ""
-			(at 0 0 0)
+			(at 0 0 180)
 			(layer "F.Fab")
 			(hide yes)
@@
 			)
 		)
+		(property "KiLib_Generator" "SMD_2terminal_chip_molded"
+			(at 0 0 180)
+			(layer "F.SilkS")
+			(hide yes)
+			(effects
+				(font
+					(size 1 1)
+					(thickness 0.15)
+				)
+			)
+		)
 		(attr smd)
 		(duplicate_pad_numbers_are_jumpers no)
@@
 		)
 		(fp_text user "${REFERENCE}"
-			(at -0.02 0.22 0)
+			(at 0 0 180)
 			(layer "F.Fab")
 			(effects
@@
 		)
 		(embedded_fonts no)
-		(model "${KICAD9_3DMODEL_DIR}/Resistor_SMD.3dshapes/R_0603_1608Metric.step"
+		(model "${KICAD10_3DMODEL_DIR}/Resistor_SMD.3dshapes/R_0603_1608Metric.step"
 			(offset
 				(xyz 0 0 0)
@@
 		(embedded_fonts no)
 	)
-	(footprint "SOIC-8_5.3x5.3mm_P1.27mm"
+	(footprint "Package_SO:SOIC-8_5.3x5.3mm_P1.27mm"
 		(layer "F.Cu")
 		(at 174.89 104.2625)
-		(descr "SOIC, 8 Pin (JEITA/EIAJ ED-7311-19 variation 08-001-BBA and Atmel/Microchip, 208 mils width, https://www.jeita.or.jp/japanese/standard/book/ED-7311-19/#target/page_no=21, https://ww1.microchip.com/downloads/en/DeviceDoc/20005045C.pdf#page=23, https://ww1.microchip.com/downloads/en/DeviceDoc/doc2535.pdf#page=162), generated with kicad-footprint-generator ipc_gullwing_generator.py")
+		(descr "SOIC, 8 Pin (JEITA/EIAJ ED-7311-19 variation 08-001-BBA and Atmel/Microchip, 208 mils width, https://www.jeita.or.jp/japanese/standard/book/ED-7311-19/#target/page_no=21, https://ww1.microchip.com/downloads/en/DeviceDoc/20005045C.pdf#page=23, https://ww1.microchip.com/downloads/en/DeviceDoc/doc2535.pdf#page=162)")
 		(tags "SOIC SO P-SOP SOP SOP-8 SO SO-8 8S2 S2AE/F K04-056 CASE-751BE SO8W 8-Pin-SOIC PSA W8-2 W8-4 W8MS-1 FPT-8P-M08")
 		(property "Reference" "U4"
@@
 			)
 		)
+		(property "KiLib_Generator" "package/gullwing"
+			(at 0 0 0)
+			(layer "F.SilkS")
+			(hide yes)
+			(effects
+				(font
+					(size 1 1)
+					(thickness 0.15)
+				)
+			)
+		)
 		(attr smd)
 		(duplicate_pad_numbers_are_jumpers no)
@@
 		)
 		(embedded_fonts no)
-		(model "${KICAD9_3DMODEL_DIR}/Package_SO.3dshapes/SOIC-8_5.3x5.3mm_P1.27mm.step"
+		(model "${KICAD10_3DMODEL_DIR}/Package_SO.3dshapes/SOIC-8_5.3x5.3mm_P1.27mm.step"
 			(offset
 				(xyz 0 0 0)
@@
 		)
 	)
-	(footprint "C_0603_1608Metric"
+	(footprint "Capacitor_SMD:C_0603_1608Metric"
 		(layer "F.Cu")
 		(at 162.8 85.94 180)
-		(descr "Capacitor SMD 0603 (1608 Metric), square (rectangular) end terminal, IPC-7351 nominal, (Body size source: IPC-SM-782 page 76, https://www.pcb-3d.com/wordpress/wp-content/uploads/ipc-sm-782a_amendment_1_and_2.pdf), generated with kicad-footprint-generator")
+		(descr "Capacitor SMD 0603 (1608 Metric), square (rectangular) end terminal, IPC-7351 nominal, (Body size source: IPC-SM-782 page 76, https://www.pcb-3d.com/wordpress/wp-content/uploads/ipc-sm-782a_amendment_1_and_2.pdf)")
 		(tags "capacitor")
 		(property "Reference" "C19"
-			(at 0 -1.43 0)
+			(at 0 -1.43 180)
 			(layer "F.SilkS")
 			(effects
@@
 		)
 		(property "Value" "100nF"
-			(at 0 1.43 0)
+			(at 0 1.43 180)
 			(layer "F.Fab")
 			(effects
@@
 		)
 		(property "Datasheet" ""
-			(at 0 0 0)
+			(at 0 0 180)
 			(layer "F.Fab")
 			(hide yes)
@@
 		)
 		(property "Description" ""
-			(at 0 0 0)
+			(at 0 0 180)
 			(layer "F.Fab")
 			(hide yes)
@@
 			)
 		)
+		(property "KiLib_Generator" "SMD_2terminal_chip_molded"
+			(at 0 0 180)
+			(layer "F.SilkS")
+			(hide yes)
+			(effects
+				(font
+					(size 1 1)
+					(thickness 0.15)
+				)
+			)
+		)
 		(attr smd)
 		(duplicate_pad_numbers_are_jumpers no)
@@
 		)
 		(fp_text user "${REFERENCE}"
-			(at 0 0 0)
+			(at 0 0 180)
 			(layer "F.Fab")
 			(effects
@@
 		)
 		(embedded_fonts no)
-		(model "${KICAD9_3DMODEL_DIR}/Capacitor_SMD.3dshapes/C_0603_1608Metric.step"
+		(model "${KICAD10_3DMODEL_DIR}/Capacitor_SMD.3dshapes/C_0603_1608Metric.step"
 			(offset
 				(xyz 0 0 0)
@@
 		)
 	)
-	(footprint "R_0603_1608Metric"
+	(footprint "Resistor_SMD:R_0603_1608Metric"
 		(layer "F.Cu")
 		(at 167.22 85.86)
-		(descr "Resistor SMD 0603 (1608 Metric), square (rectangular) end terminal, IPC-7351 nominal, (Body size source: IPC-SM-782 page 72, https://www.pcb-3d.com/wordpress/wp-content/uploads/ipc-sm-782a_amendment_1_and_2.pdf), generated with kicad-footprint-generator")
+		(descr "Resistor SMD 0603 (1608 Metric), square (rectangular) end terminal, IPC-7351 nominal, (Body size source: IPC-SM-782 page 72, https://www.pcb-3d.com/wordpress/wp-content/uploads/ipc-sm-782a_amendment_1_and_2.pdf)")
 		(tags "resistor")
 		(property "Reference" "R11"
@@
 			)
 		)
+		(property "KiLib_Generator" "SMD_2terminal_chip_molded"
+			(at 0 0 0)
+			(layer "F.SilkS")
+			(hide yes)
+			(effects
+				(font
+					(size 1 1)
+					(thickness 0.15)
+				)
+			)
+		)
 		(attr smd)
 		(duplicate_pad_numbers_are_jumpers no)
@@
 		)
 		(embedded_fonts no)
-		(model "${KICAD9_3DMODEL_DIR}/Resistor_SMD.3dshapes/R_0603_1608Metric.step"
+		(model "${KICAD10_3DMODEL_DIR}/Resistor_SMD.3dshapes/R_0603_1608Metric.step"
 			(offset
 				(xyz 0 0 0)
@@
 		)
 	)
-	(footprint "C_0402_1005Metric"
+	(footprint "Capacitor_SMD:C_0402_1005Metric"
 		(layer "F.Cu")
 		(at 151.94 87.05 -45)
-		(descr "Capacitor SMD 0402 (1005 Metric), square (rectangular) end terminal, IPC-7351 nominal, (Body size source: IPC-SM-782 page 76, https://www.pcb-3d.com/wordpress/wp-content/uploads/ipc-sm-782a_amendment_1_and_2.pdf), generated with kicad-footprint-generator")
+		(descr "Capacitor SMD 0402 (1005 Metric), square (rectangular) end terminal, IPC-7351 nominal, (Body size source: IPC-SM-782 page 76, https://www.pcb-3d.com/wordpress/wp-content/uploads/ipc-sm-782a_amendment_1_and_2.pdf)")
 		(tags "capacitor")
 		(property "Reference" "C21"
-			(at 0 -1.16 135)
+			(at 0 -1.16 315)
 			(layer "F.SilkS")
 			(effects
@@
 		)
 		(property "Value" "12pF"
-			(at 0 1.16 135)
+			(at 0 1.16 315)
 			(layer "F.Fab")
-			(hide yes)
 			(effects
 				(font
@@
 		)
 		(property "Datasheet" ""
-			(at 0 0 135)
+			(at 0 0 315)
 			(layer "F.Fab")
 			(hide yes)
@@
 		)
 		(property "Description" ""
-			(at 0 0 135)
+			(at 0 0 315)
 			(layer "F.Fab")
 			(hide yes)
@@
 			)
 		)
+		(property "KiLib_Generator" "SMD_2terminal_chip_molded"
+			(at 0 0 315)
+			(layer "F.SilkS")
+			(hide yes)
+			(effects
+				(font
+					(size 1 1)
+					(thickness 0.15)
+				)
+			)
+		)
 		(attr smd)
 		(duplicate_pad_numbers_are_jumpers no)
@@
 		)
 		(fp_text user "${REFERENCE}"
-			(at 0 0 135)
+			(at 0 0 315)
 			(layer "F.Fab")
 			(effects
@@
 		)
 		(embedded_fonts no)
-		(model "${KICAD9_3DMODEL_DIR}/Capacitor_SMD.3dshapes/C_0402_1005Metric.step"
+		(model "${KICAD10_3DMODEL_DIR}/Capacitor_SMD.3dshapes/C_0402_1005Metric.step"
 			(offset
 				(xyz 0 0 0)

Commit message: Carrier: S5 pull-ups, unused-pin test-pad breakouts, value-only silk
- Add R44-R49 (100k) pull-ups/pull-downs for the BMC<->SoC link, SFC_IO2/IO3 and NOR CE
- Break out unused U15 P11-P17, U8 SPIIO7/MTMS/console UART and U12 spare VBUS to 1.0mm test pads
- Tie J4 SHIELD and J6 G to GND; no-connect the remaining unused pins (ERC pin_not_connected 30 -> 0)
- Silkscreen: show values/part names instead of references for R/C/U/L/D/Q/SW/JP (J refs kept)
- Refill zones; remove stray no-net track segments
- Interposer: SFC shared-bus pinout/schematic updates
Parts:
- removed U4: W25Q32JVSS, Package_SO:SOIC-8_5.3x5.3mm_P1.27mm
- IC1: footprint teacup:QFN35P900X900X90-89N-D -> teacup-interposer:QFN35P900X900X90-89N-D
- J1: footprint DIMM-DDR4 -> teacup-interposer:DIMM-DDR4
- TP1, TP2, TP3, TP4, TP5, TP6, TP7: footprint TestPoint_Pad_2.0x2.0mm -> TestPoint:TestPoint_Pad_2.0x2.0mm
- moved TP7 16.5 mm to (102.0, 94.4)
- moved TP6 15.4 mm to (102.1, 100.0)
- turned C20 to 135 degrees
Connections:
- C20 pad 1: GND -> /EXCLK_I
- C20 pad 2: /EXCLK_I -> GND
- IC1 pad 45: SSI0_CE0 -> SFC_CS
- IC1 pad 46: SSI0_DR -> SFC_IO1
- IC1 pad 47: SSI0_DT -> SFC_IO0
- IC1 pad 48: SSI0_CLK -> SFC_CLK
Routing:
- net SSI0_CE0: track 63.0 -> 0.00 mm, vias 4 -> 0
- net SFC_CLK: track 0.00 -> 60.1 mm, vias 0 -> 2
- net SFC_IO0: track 0.00 -> 59.8 mm, vias 0 -> 2
- net SSI0_DT: track 58.4 -> 0.00 mm, vias 3 -> 0
- net SFC_IO1: track 0.00 -> 57.6 mm, vias 0 -> 2
- net SFC_CS: track 0.00 -> 56.8 mm, vias 0 -> 3
- net SSI0_DR: track 53.9 -> 0.00 mm, vias 2 -> 0
- net SSI0_CLK: track 52.4 -> 0.00 mm, vias 4 -> 0
- net +1V8: track 174.3 -> 140.1 mm, vias 13 -> 12
- net USBA_HOST_DM: track 56.3 -> 81.4 mm, vias 4 -> 6
- net USBA_HOST_DP: track 56.0 -> 73.8 mm, vias 2 -> 6
- net GND: track 82.6 -> 99.8 mm
- net SPARE_P181: track 57.9 -> 62.1 mm
- net SPARE_P180: track 61.0 -> 64.8 mm
- net SPARE_P177: track 41.8 -> 44.9 mm
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- added copper zone on In1.Cu, net GND
- added copper zone on In2.Cu, net GND
