File: hw/interposer_t41/teacup-interposer-t41.kicad_sch (KiCad schematic)
At the start: 31 parts, among them J1 DIMM-DDR4, U11 T41, U7 GD25Q127CSIG, Y1 24 MHz

Commit message: Backfill MPN/Manufacturer fields on carrier and interposer schematics
Placed symbol instances only carried Reference/Value/Footprint; MPN and
Manufacturer were never propagated from the library cache, so BOM export
had a blank MPN column for every part. Fills in MPN (and Manufacturer
where unambiguous) for the 32 parts whose Value string is already a real
manufacturer part number - ICs, diodes, MOSFETs, switches, and specific
connectors - across the carrier, T31ZX interposer, and T41 interposer.
Generic passives, headers, and jumpers are left untouched since their
Value is a spec, not a part number.

ERC-neutral: 426/175/169 violations before and after on the three files.
Parts:
- U11: MPN (none) -> T41; Manufacturer (none) -> Ingenic Semiconductor
- U7: MPN (none) -> GD25Q127CSIG; Manufacturer (none) -> GigaDevice Semiconductor
Changed lines of the file:
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@@
 		(property "Value" "T41" (at 203.2 330.2 0) (effects (font (size 1.27 1.27))))
 		(property "Footprint" "teacup-interposer-t41:T41_QFN96" (at 203.2 228.6 0) (effects (font (size 1.27 1.27)) hide))
+		(property "MPN" "T41" (at 203.2 228.6 0) (effects (font (size 1.27 1.27)) hide))
+		(property "Manufacturer" "Ingenic Semiconductor" (at 203.2 228.6 0) (effects (font (size 1.27 1.27)) hide))
 	)
 	(symbol (lib_id "power:GND") (at 236.22 289.56 90) (unit 1)
@@
 		(property "Value" "GD25Q127CSIG" (at 88.9 64.77 0) (effects (font (size 1.27 1.27))))
 		(property "Footprint" "Package_SO:SOIC-8_5.3x5.3mm_P1.27mm" (at 88.9 57.15 0) (effects (font (size 1.27 1.27)) hide))
+		(property "MPN" "GD25Q127CSIG" (at 88.9 57.15 0) (effects (font (size 1.27 1.27)) hide))
+		(property "Manufacturer" "GigaDevice Semiconductor" (at 88.9 57.15 0) (effects (font (size 1.27 1.27)) hide))
 	)
 	(symbol (lib_id "power:GND") (at 88.9 69.85 0) (unit 1)
